File: pcb/microfloat.brd (EAGLE design)
At the start: 76.2 x 66 mm, 107 parts, among them J1 503182-1852, J11 JTAG-MINI, J12 XT-60BATT_LABEL, J2 USB4105_REVA, J9 1909763-1, U1 BME280, U2 ICM-42688-P, U3 MAX13237EETE, U4 NEO-M8N-0, U5 TXB0104PWR, U6 ATSAMD51J19A-AUT, U7 Value, Y1 32.768kHz

Commit message: changes changes changes
Parts:
- removed PS3: LMZ14201HTZX/NOPB, microfloat:CONV_LMZ14201HTZX/NOPB
- removed R27, R28: 0, rcl:R0603
- added C42, C43, C44: 47uF, rcl:C0603
- added L2: 380hm, RoboJackets-Inductors:0805
- added U8: Value, microfloat:RPK0013A-MFG
- C28, C30: value 10uF -> 47uF
- C29: value 4700pF -> 47uF
- C31: value 100uF -> 47uF
- R22: value 100k -> 7.5k
- R23: value 1.2k -> 7.5k
- R24: value 100 -> 7.5k
- R25: value 6.49k -> 100k
- R26: value 34k -> 100k
- moved R26 97.2 mm to (-34.0, -74.0), flipped to the top, turned to 0 degrees
- moved R25 93.5 mm to (-34.0, -69.0), flipped to the top
- moved R24 82.9 mm to (-34.0, -49.0), flipped to the top
- moved R23 78.0 mm to (-34.0, -44.0), flipped to the top, turned to 0 degrees
- moved R22 76.7 mm to (-34.0, -39.0), flipped to the top
- moved C31 68.5 mm to (-33.0, -29.0), flipped to the top, turned to 0 degrees
- moved C30 62.6 mm to (-33.0, -24.0), flipped to the top
- moved C29 62.3 mm to (-33.0, -19.0), flipped to the top, turned to 0 degrees
- moved C28 58.3 mm to (-33.0, -14.0), flipped to the top, turned to 0 degrees
Connections:
- removed net N$21: PS3.3, R23.1, R24.2
- new net N$30: C44.2, L2.1, U8.12
- new net N$31: C44.1, U8.4
- new net RREF+: J15.1, R26.1
- new net RREF-: J15.4
- new net RSENSE+: J15.2, R25.1
- new net RSENSE-: J15.3
- net +12V: now also C42.1, C43.1, L2.2, R22.2, R23.1; no longer C30.1, C31.1, PS3.7, R26.2
- net +3V3: now also R25.2, R26.2; no longer R27.2, R28.2
- net GND: now also C30.2, C42.2, C43.2, U8.1, U8.11, U8.13, U8.6; no longer PS3.4, PS3.8, R25.1
- net LEVEL: no longer J15.1, J15.2, J15.3, J15.4, R27.1, R28.1
- net N$22: now also R23.2, U8.8; no longer PS3.2, R22.2
- net N$23: now also R22.1, R24.2, U8.7; no longer C29.1, PS3.5
- net N$24: now also C31.1, U8.5; no longer C30.2, PS3.6, R25.2, R26.1
- net VBATT: now also C29.1, C30.1, U8.10, U8.2, U8.9; no longer PS3.1, R22.1, R23.2
Routing:
- net GND: track 248.8 -> 211.0 mm, vias 75 -> 65
- net LEVEL: track 47.5 -> 30.4 mm
- net VBATT: track 39.6 -> 24.5 mm, vias 7 -> 4
- net N$24: track 9.89 -> 0.00 mm, vias 1 -> 0
- net +12V: track 12.1 -> 2.74 mm, vias 2 -> 1
- net N$22: track 6.60 -> 0.00 mm, vias 1 -> 0
- net N$21: track 6.22 -> 0.00 mm, vias 1 -> 0
- net N$23: track 4.31 -> 0.00 mm, vias 1 -> 0
- net +3V3: track 39.5 -> 36.8 mm, vias 15 -> 13

Commit message: CHANGES CHANGES CHANGES
Parts:
- removed C26: 1nF, rcl:C0603
- removed C27, C28, C29, C30, C31, C42, C43, C44: 47uF, rcl:C0603
- removed C40: 0.1uF, rcl:C0603
- removed C41: 1uF, rcl:C0603
- removed D2, D3: 30V, microfloat:MICROSMP
- removed J12: XT-60BATT_LABEL, microfloat:XT-60
- removed PS1, PS2: LMZ14201HTZX/NOPB, microfloat:CONV_LMZ14201HTZX/NOPB
- removed R14: 110k, rcl:R0603
- removed R15, R20: 1.07k, rcl:R0603
- removed R16: 5.62k, rcl:R0603
- removed R17: 133K, rcl:R0603
- removed R18: 68.1k, rcl:R0603
- removed R19, R22, R23, R24: 7.5k, rcl:R0603
- removed R21: 6.98k, rcl:R0603
- removed U$19: (no value), RoboJackets-Fuses:3568
- added C53: 33uF, rcl:C0603
- added C54, C58: 100nF, rcl:C0603
- added C55, C56, C59, C60: 22uF, rcl:C0603
- added C57: 10uF, rcl:C0603
- added CR1, CR2: STTH2L06A, microfloat:SMA_STM
- added L3: 12uH, RoboJackets-Inductors:0805
- added L5: 6.471uH, RoboJackets-Inductors:0805
- added L6: 13uH, RoboJackets-Inductors:0805
- added R31, R33: 100k, rcl:R0603
- added R32: 5.23k, rcl:R0603
- added R34: 11k, rcl:R0603
- added U12, U13: TPS54308DDCT, microfloat:SOT95P280X110-6N
- added U9: ATSAMD51N20A-AUT, microfloat:QFP50P1600X1600X120-100N
- C17: value 10uF -> 33uF
- C18: value 470pF -> 100nF
- C19, C20, C24: value 10uF -> 22uF
- C21: value 10nF -> 10uF
- C22: value 1nF -> 33uF
- C23: value 100uF -> 100nF
- C25: value 10nF -> 22uF
- L2: value 380hm -> 12uH
- R10: value 118k -> 100k
- R11: value 150k -> 13.7k
- R12: value 68.1k -> 100k
- R13: value 7.5k -> 13.7k
- U7: value Value -> TPS54308DDCT; device microfloat:SIL0008A -> microfloat:SOT95P280X110-6N
- U8: value Value -> TPS54308DDCT; device microfloat:RPK0013A-MFG -> microfloat:SOT95P280X110-6N
- moved C22 285.5 mm to (-58.0, -224.0), flipped to the top, turned to 0 degrees
- moved R13 282.7 mm to (-58.0, -219.0), flipped to the top, turned to 0 degrees
- moved R12 279.1 mm to (-52.0, -219.0), flipped to the top, turned to 0 degrees
- moved C23 278.4 mm to (-48.0, -212.0), flipped to the top, turned to 0 degrees
- moved C21 273.4 mm to (-58.0, -207.0), flipped to the top, turned to 0 degrees
- moved C25 264.6 mm to (-58.0, -229.0), flipped to the top, turned to 0 degrees
- moved C20 264.5 mm to (-58.0, -202.0), flipped to the top, turned to 0 degrees
- moved C24 253.5 mm to (-52.0, -224.0), flipped to the top, turned to 0 degrees
- moved C17 253.2 mm to (-58.0, -197.0), flipped to the top, turned to 0 degrees
- moved C19 252.6 mm to (-52.0, -197.0), flipped to the top, turned to 0 degrees
- moved R10 245.5 mm to (-52.0, -192.0), flipped to the top, turned to 0 degrees
- moved R11 245.2 mm to (-58.0, -192.0), flipped to the top, turned to 0 degrees
- moved U7 244.3 mm to (-57.0, -186.0), flipped to the top, turned to 0 degrees
- moved C18 236.9 mm to (-48.0, -185.0), flipped to the top, turned to 0 degrees
- moved U8 207.4 mm to (-57.0, -213.0)
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Connections:
- removed net N$17: PS1.3, R18.1, R19.2
- removed net N$18: PS1.2, R17.2
- removed net N$19: C25.1, PS1.5
- removed net N$20: C26.2, PS1.6, R20.2, R21.1
- removed net N$22: R23.2, U8.8
- removed net N$23: R22.1, R24.2, U8.7
- removed net N$24: C31.1, U8.5
- removed net N$28: C40.1, C41.1, U$19.P$1, U$19.P$2
- removed net N$30: C44.2, L2.1, U8.12
- removed net N$31: C44.1, U8.4
- new net N$21: U6.52
- new net N$35: C54.1, U12.6
- new net N$36: C54.2, L5.1, U12.2
- new net N$37: R31.1, R32.2, U12.4
- new net N$38: C58.1, U13.6
- new net N$39: C58.2, L6.1, U13.2
- new net N$40: R33.1, R34.2, U13.4
- new net VDDIOB: U9.25, U9.30
- net !RESET: now also U9.88; no longer U6.52
- net +12V: now also C55.1, C56.1, L5.2, R31.2; no longer C42.1, C43.1, L2.2, R22.2, R23.1
- net +3V3: now also C24.1, C25.1, L3.2, R12.2, U9.39, U9.51, U9.63, U9.77, U9.92; no longer C17.1, U7.3, U7.5
- net +5V: now also C20.1, C22.1, CR1.1, CR2.1, L2.2, R10.2, U8.3; no longer D2.K, D3.K, U7.7
- net +6V: now also C59.1, C60.1, L6.2, R33.2; no longer C26.1, C27.1, PS1.7, R21.2
- net GND: now also C22.2, C53.2, C55.2, C56.2, C57.2, C59.2, C60.2, R32.1, R34.1, U12.1, U13.1, U7.1, U9.11, U9.24, U9.31, U9.38, U9.50, U9.62, U9.76, U9.90; no longer C18.2, C23.2, C27.2, C28.2, C29.2, C30.2, C31.2, C40.2, C41.2, C42.2, C43.2, J12.GND, PS1.4, PS1.8, PS2.4, PS2.8, R15.1, R19.1, R20.1, R24.1, U7.4, U7.6, U7.9, U8.11, U8.13, U8.6
- net N$11: now also C18.1, U7.6; no longer PS2.3, R12.1, R13.2
- net N$12: now also C18.2, L2.1, U7.2; no longer R10.2, U7.8
- net N$13: now also U7.4; no longer C18.1, U7.2
- net N$14: now also C23.1, U8.6; no longer PS2.2, R14.2
- net N$15: now also C23.2, L3.1, U8.2; no longer C21.1, PS2.5
- net N$16: now also R12.1, R13.2, U8.4; no longer C22.2, PS2.6, R15.2, R16.1
- net VBATT: now also C17.1, C21.1, C53.1, C57.1, U12.3, U13.3, U7.3; no longer C20.1, C24.1, C28.1, C29.1, C30.1, J12.BATT, PS1.1, PS2.1, R12.2, R14.1, R17.1, R18.2, U$19.P$3, U$19.P$4, U8.10, U8.2, U8.9
- net VBATT_5V: now also CR2.2; no longer C22.1, C23.1, D3.A, PS2.7, R16.2
- net VBUS: now also CR1.2; no longer D2.A
- net VCCA: now also U9.12
- net VCC_CORE: now also U9.89
Routing:
- net GND: track 211.0 -> 141.3 mm, vias 65 -> 45
- net VBATT: track 24.5 -> 0.00 mm, vias 4 -> 0
- net N$20: track 23.7 -> 0.00 mm, vias 2 -> 0
- net VBATT_5V: track 18.3 -> 0.00 mm, vias 2 -> 0
- net N$16: track 16.3 -> 0.00 mm, vias 1 -> 0
- net N$19: track 14.3 -> 0.00 mm, vias 2 -> 0
- net N$17: track 9.89 -> 0.00 mm
- net +5V: track 17.9 -> 8.04 mm, vias 5 -> 2
- net N$14: track 9.73 -> 0.00 mm, vias 1 -> 0
- net N$28: track 8.49 -> 0.00 mm
- net N$11: track 7.71 -> 0.00 mm, vias 1 -> 0
- net N$13: track 6.42 -> 0.00 mm
- net N$15: track 5.31 -> 0.00 mm, vias 1 -> 0
- net N$18: track 4.62 -> 0.00 mm
- net +3V3: track 36.8 -> 32.7 mm, vias 13 -> 11
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
Commit message: changessssssssss, mcu pinout
Parts:
- removed U6: ATSAMD51J19A-AUT, microfloat:QFP50P1200X1200X120-64N
- added C26: 0.1uF, rcl:C0603
- added F1: 0.5A, microfloat:F1206
- added F2: 2A, microfloat:F1206
- added F3: 0.25A, microfloat:F1206
- added F4: 0.6A, microfloat:F1206
- added R14, R15, R19: 10k, rcl:R0603
- added R16, R17, R18: 100k, rcl:R0603
- C6: value 10 nF -> 0.1uF
- R1: value 10k -> 100k
Connections:
- removed net CS_CD: J1.2
- removed net CS_SD: U6.15
- removed net LEVEL: U6.3
- removed net N$21: U6.52
- removed net R_IN: U3.5, U6.60
- removed net T_IN: U3.8, U6.59
- removed net VDDIOB: U9.25, U9.30
- removed net VSW: U6.55
- new net MODEM_R_IN: U3.5, U9.56
- new net MODEM_T_IN: U3.8, U9.57
- new net N$17: C55.1, C56.1, F2.1, L5.2, R31.2
- new net N$18: C59.1, C60.1, F3.1, L6.2, R33.2
- new net N$19: C19.1, C20.1, F4.1, L2.2, R10.2
- new net N$20: C24.1, C25.1, F1.1, L3.2, R12.2
- new net N$25: R14.2, R15.2, R16.2, R17.2, R18.2
- new net SD_CD: J1.2, R14.1, U9.19
- new net SD_CK: J1.5, U9.33
- new net SD_CMD: J1.3, R15.1, U9.26
- new net SD_DATA0: J1.7, R17.1, U9.27
- new net SD_DATA1: J1.8, R18.1, U9.28
- new net SD_DATA2: J1.1, R16.1, U9.29
- net !RESET_N: now also U9.72; no longer U6.19
- net !SX-NRESET: now also U9.68; no longer U6.44
- net +12V: now also F2.2; no longer C55.1, C56.1, L5.2, R31.2
- net +3V3: now also C26.1, F1.2, J1.4, R19.1, U9.25, U9.30; no longer C24.1, C25.1, L3.2, R12.2, U6.21, U6.34, U6.48, U6.56
- net +5V: now also F4.2; no longer C19.1, C20.1, L2.2, R10.2
- net +6V: now also F3.2; no longer C59.1, C60.1, L6.2, R33.2
- net ANT_SW: now also U9.69; no longer U6.43
- net CO2: no longer U6.4
- net CS_GPS: now also U9.48; no longer U6.42
- net CS_IMU: now also U9.55; no longer U6.38
- net CS_PHT: now also U9.83; no longer U6.32
- net CS_RAD: now also U9.49; no longer U6.41
- net D_N: now also U9.74; no longer U6.45
- net D_P: now also U9.75; no longer U6.46
- net GND: now also C26.2, J1.6; no longer U6.22, U6.33, U6.47, U6.54, U6.7
- net LEAK: now also U9.36; no longer U6.18
- net LNA_EN: now also U9.73; no longer U6.28
- net MISO_1: now also U9.82; no longer U6.31
- net MISO_2: now also U9.54; no longer J1.7, U6.37
- net MOSI_1: now also U9.80; no longer U6.29
- net MOSI_2: now also U9.52; no longer J1.3, U6.35
- net RAD_BUSY: no longer U6.27
- net SCLK_1: now also U9.81; no longer U6.30
- net SCLK_2: now also U9.53; no longer J1.5, U6.36
- net SOLENOID: now also U9.37; no longer U6.20
- net SWCLK: now also R19.2, U9.93; no longer U6.57
- net SWDIO: now also U9.94; no longer U6.58
- net UART_RX_CTD_A: now also U9.34; no longer U6.25
- net UART_RX_M_A: now also U9.64; no longer U6.39
- net UART_RX_PH: now also U9.46; no longer U6.16
- net UART_TX_CTD_A: now also U9.35; no longer U6.26
- net UART_TX_M_A: now also U9.65; no longer U6.40
- net UART_TX_PH: now also U9.47; no longer U6.17
- net VCCA: no longer U6.8
- net VCC_CORE: no longer U6.53
- net XIN32: no longer U6.1
- net XOUT32: no longer U6.2
Routing:
- net LEVEL: track 30.4 -> 0.00 mm, vias 1 -> 0
- net UART_TX_PH: track 20.9 -> 0.00 mm
- net UART_RX_PH: track 15.4 -> 0.00 mm
- net CO2: track 26.8 -> 15.3 mm
- net SOLENOID: track 20.7 -> 11.5 mm
- net MOSI_2: track 49.9 -> 40.8 mm
- net GND: track 141.3 -> 136.1 mm, vias 45 -> 42
- net SCLK_1: track 35.3 -> 31.0 mm
- net CS_PHT: track 8.68 -> 4.38 mm
- net MISO_1: track 36.8 -> 32.5 mm
- net T_IN: track 3.39 -> 0.00 mm
- net R_IN: track 3.27 -> 0.00 mm
- net SCLK_2: track 48.5 -> 45.3 mm
- net MOSI_1: track 39.3 -> 36.4 mm
- net MODEM_T_IN: track 0.00 -> 2.62 mm
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
Commit message: Power wee
Parts:
- removed CR1, CR2: STTH2L06A, microfloat:SMA_STM
- added C27, C28: 10uF, rcl:C0603
- added R20, R21, R22, R23, R24: 100k, rcl:R0603
- added U$12, U$13, U$19, U$20, U$21, U$24, U$6, U$7, U$8, U$9: TEST_POINT, microfloat:TEST_POINT
- added U6: LTC4419CMSEPBF, microfloat:MSE_12_ADI
- C22: value 33uF -> 22uF
- L3: value 12uH -> 3.9uH
- R13: value 13.7k -> 22k
Connections:
- removed net VBATT_5V: CR2.2
- new net +5V_BATT: F4.2, U$9.P$1
- new net N$21: R20.1, R21.2, U6.4
- new net N$22: R21.1, R22.2, U6.3
- new net N$23: R23.1, R24.2, U6.10
- new net N$24: C27.1, R20.2, U6.1
- new net N$26: C28.1, R23.2, U6.12
- new net N$28: U$12.P$1, U6.8
- new net N$29: U6.9
- net +12V: now also U$7.P$1
- net +3V3: now also U$6.P$1
- net +5V: no longer CR1.1, CR2.1, F4.2
- net +6V: now also U$8.P$1
- net GND: now also C27.2, C28.2, R22.1, R24.1, U$13.P$1, U$19.P$1, U$20.P$1, U$21.P$1, U$24.P$1, U6.5, U6.EPAD
- net VBUS: no longer CR1.2

Commit message: more schematic changes (conn fix, solenoid fix, etc)
Parts:
- removed D1: 30V, microfloat:MICROSMP
- removed J10, J13, J15, J16, J17, J18, J7, J8: (no value), microfloat:MOLEX_NANOFIT_SMD_RIGHTANGLE_04
- added CR1: VSKY20401608-G4-08, microfloat:CLP1608-2L_VIS
- added F5: 0.5A, microfloat:F1206
- added J3, J4: 1054291110, microfloat:CON_1054291110_MOL
- added J5: 1054291116, microfloat:CON_1054291116_MOL
- added R27: 10, rcl:R0603
- added R28: 100k, rcl:R0603
- added U$27: GSOT04-E3-08, microfloat:SOT-23-3
- added U$29: TEST_POINT, microfloat:TEST_POINT
- C10, C11, C12, C7, C8, C9: value 0.1 uF -> 0.2 uF
- R25: value 100k -> 652
- R26: value 100k -> 1k'
- R3: value 240 -> 100k
- U$1: value SQ2364EES-T1_GE3 -> SQ2348ES-T1_GE3
- moved R3 418.9 mm to (-87.6, -387.4), flipped to the top, turned to 0 degrees
- moved U$1 386.7 mm to (-81.3, -369.6), turned to 0 degrees
Connections:
- net CO2 renamed CO2_OUT
- removed net +5V_BATT: F4.2, U$9.P$1
- removed net AGND: J7.4, R7.1
- removed net N$27: D1.A, J14.1, U$1.3
- new net CO2_IN: J3.1, R6.2
- new net SOL_TRIG: CR1.2, J14.1, J5.13, U$1.3
- new net VBATT_5V: C28.1, F4.2, R23.2, U$9.P$1, U6.12
- net +12V: now also CR1.1, J5.14; no longer D1.K
- net +3V3: now also J4.9, R28.1; no longer J8.1, U3.9
- net +5V: now also J3.9, U6.9; no longer J13.1
- net +6V: now also J3.10; no longer J7.1
- net GND: now also J3.2, J3.3, J3.4, J3.5, J3.6, J3.7, J3.8, J5.15, J5.5, J5.7, R7.1, U$27.3, U3.9; no longer J10.3, J13.4, J16.1, J17.2, J17.4, J18.2, J18.4, J7.2, J8.4
- net LEAK: no longer R3.2
- net N$1: now also R28.2, U5.8; no longer J7.3, R6.2
- net N$24: now also R27.1, U$1.1; no longer C27.1, R20.2, U6.1
- net N$26: now also C27.1, F5.2, R20.2, U6.1; no longer C28.1, R23.2, U6.12
- net N$29: now also J5.6; no longer U6.9
- net PROBE: now also J4.7, J4.8, J5.11, J5.12; no longer J17.1, J17.3, J18.1, J18.3
- net RREF+: now also J5.1; no longer J15.1
- net RREF-: now also J5.4; no longer J15.4
- net RSENSE+: now also J5.2; no longer J15.2
- net RSENSE-: now also J5.3; no longer J15.3
- net R_OUT: now also J4.3; no longer J16.3
- net SOLENOID: now also R27.2, R3.2, U$27.1; no longer U$1.1
- net T_OUT: now also J4.4; no longer J16.2
- net UART_RX_CTD_B: now also J4.6; no longer J13.3
- net UART_RX_M_B: now also J5.10; no longer J10.2
- net UART_RX_PH: now also J4.1; no longer J8.2
- net UART_TX_CTD_B: now also J4.5; no longer J13.2
- net UART_TX_M_B: now also J5.9; no longer J10.1
- net UART_TX_PH: now also J4.2; no longer J8.3
- net VBATT: now also J5.16
- net VBUS: now also F5.1, U$29.P$1
Routing:
- net GND: track 136.1 -> 112.5 mm, vias 42 -> 35
- net PROBE: track 17.8 -> 4.61 mm, vias 2 -> 1
- net SOLENOID: track 11.5 -> 0.00 mm
- net +5V: track 8.04 -> 1.19 mm, vias 2 -> 1
- net N$1: track 6.48 -> 0.00 mm, vias 1 -> 0
- net N$27: track 5.59 -> 0.00 mm, vias 1 -> 0
- net AGND: track 4.57 -> 0.00 mm, vias 1 -> 0
- net CO2_IN: track 0.00 -> 4.41 mm, vias 0 -> 1
- net UART_RX_M_B: track 14.2 -> 11.3 mm
- net +12V: track 2.74 -> 0.00 mm, vias 1 -> 0
- net UART_TX_M_B: track 18.1 -> 15.4 mm
- net LEAK: track 11.2 -> 9.03 mm
- net +6V: track 2.20 -> 0.00 mm, vias 1 -> 0
- net T_OUT: track 17.2 -> 15.8 mm
- net UART_TX_CTD_B: track 12.2 -> 11.1 mm
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
Commit message: Improved signal buffering on connectors and hi Asha
Parts:
- added C29, C30, C40: 1.0 uF, rcl:C0603
- added C31: 10uF, rcl:C0603
- added R29: 560k, rcl:R0603
- added R30: 100k, rcl:R0603
- added U$31, U$32: TEST_POINT, microfloat:TEST_POINT
- C1, C2: value 100 nF -> 0.1 uF
- C5: value 10 nF -> 0.01 uF
- R20: value 100k -> 390k
- R21: value 100k -> 68k
- R22: value 100k -> 43k
- R23: value 100k -> 910k
- R24: value 100k -> 82k
- T1: value (none) -> MMBT3906
Connections:
- removed net N$29: J5.6
- new net BATT_MEASURE: R29.1, R30.2, U9.100
- new net GND1: C11.2, C12.2, C29.2, C30.2, C8.2
- new net IMU_INT: U2.4, U9.70
- new net N$30: J4.11
- net +3V3: now also C29.1, C30.1, C40.1
- net +5V: now also C31.1, J3.5, U$31.P$1; no longer J3.9
- net GND: now also C31.2, C40.2, J3.11, J3.12, J3.9, J4.12, J5.12, J5.13, J5.17, J5.18, J5.4, R30.1, U$32.P$1; no longer C11.2, C12.2, C8.2, J3.5, J5.7
- net PROBE: now also J4.10, J4.5, J5.3; no longer J4.7, J4.8, J5.12
- net RREF-: now also J5.9; no longer J5.4
- net RSENSE-: now also J5.10; no longer J5.3
- net SOL_TRIG: now also J5.6; no longer J5.13
- net UART_RX_M_B: now also J5.7; no longer J5.10
- net UART_TX_CTD_B: now also J4.7; no longer J4.5
- net UART_TX_M_B: now also J5.8; no longer J5.9
- net VBATT: now also R29.2
Routing:
- net GND1: track 0.00 -> 13.7 mm, vias 0 -> 2
- net GND: track 112.5 -> 98.8 mm, vias 35 -> 33

Commit message: ADC resolved
Connections:
- net BATT_MEASURE: now also U9.15; no longer U9.100
- net CO2_OUT: now also U9.13
- net RREF+: now also U9.97
- net RSENSE+: now also U9.99
Changed lines of the file:
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@@
 <wire x1="-8" y1="39" x2="-7.976121875" y2="38.976121875" width="0.254" layer="16"/>
 <wire x1="-7.976121875" y1="38.976121875" x2="-7.976121875" y2="37.525" width="0.254" layer="16"/>
+<contactref element="U9" pad="13"/>
+<wire x1="-9.32388125" y1="36.785" x2="-52.67" y2="-65" width="0" layer="19" extent="1-16"/>
 </signal>
 <signal name="UART_RX_PH">
@@
 <contactref element="R25" pad="1"/>
 <contactref element="J5" pad="2"/>
+<contactref element="U9" pad="99"/>
 <wire x1="-34.85" y1="-69" x2="-106.64" y2="-401.32" width="0" layer="19" extent="1-1"/>
+<wire x1="-50.5" y1="-57.33" x2="-34.85" y2="-69" width="0" layer="19" extent="1-1"/>
 </signal>
 <signal name="RREF+">
 <contactref element="R26" pad="1"/>
 <contactref element="J5" pad="1"/>
+<contactref element="U9" pad="97"/>
 <wire x1="-34.85" y1="-74" x2="-104.14" y2="-401.32" width="0" layer="19" extent="1-1"/>
+<wire x1="-49.5" y1="-57.33" x2="-34.85" y2="-74" width="0" layer="19" extent="1-1"/>
 </signal>
 <signal name="N$35">
@@
 <contactref element="R30" pad="2"/>
 <contactref element="R29" pad="1"/>
-<contactref element="U9" pad="100"/>
-<wire x1="-124.04" y1="-458.47" x2="-51" y2="-57.33" width="0" layer="19" extent="1-1"/>
+<contactref element="U9" pad="15"/>
+<wire x1="-124.04" y1="-458.47" x2="-52.67" y2="-66" width="0" layer="19" extent="1-1"/>
 <wire x1="-122.34" y1="-463.55" x2="-124.04" y2="-458.47" width="0" layer="19" extent="1-1"/>
 </signal>
