File: pcb/microfloat.brd (EAGLE design)
At the start: 76.2 x 66 mm, 135 parts, among them J1 503182-1852, J11 JTAG-MINI, J2 USB4105_REVA, J3 1054291110, J4 1054291110, J5 1054291116, J9 1909763-1, T1 MMBT3906, U1 BME280, U12 TPS54308DDCT, U13 TPS54308DDCT, U2 ICM-42688-P, U3 MAX13237EETE, U4 NEO-M8N-0, U5 TXB0104PWR, U6 LTC4419CMSEPBF, U7 TPS54308DDCT, U8 TPS54308DDCT, U9 ATSAMD51N20A-AUT, Y1 32.768kHz

Commit message: More changes
Parts:
- removed J14: (no value), microfloat:MOLEX_NANOFIT_SMD_RIGHTANGLE_02
Connections:
- new net READY: U3.14, U9.9
- net +12V: no longer J14.2
- net GND: now also J1.P1, J1.P2, J1.P3, J1.P4, J1.P5
- net SOL_TRIG: no longer J14.1
Changed lines of the file:
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@@
 <attribute name="VALUE" x="50.579253125" y="35.325334375" size="1.27" layer="28" rot="MR150.5"/>
-</element>
-<element name="J14" library="microfloat" package="MOLEX_NANOFIT_SMD_RIGHTANGLE_02" value="" x="12.3" y="9.3" smashed="yes" rot="MR0">
-<attribute name="MPN" value="1054301202" x="23.3" y="34.3" size="1.778" layer="28" rot="MR0" display="off"/>
-<attribute name="NAME" x="12.3" y="11.84" size="0.8128" layer="26" font="vector" rot="MR0" align="bottom-center"/>
 </element>
 <element name="C32" library="rcl" library_urn="urn:adsk.eagle:library:334" package="C0603" package3d_urn="urn:adsk.eagle:package:23616/2" value="0.1uF" x="18.2" y="34.1" smashed="yes" rot="MR270">
@@
 <contactref element="J5" pad="12"/>
 <contactref element="J5" pad="13"/>
+<contactref element="J1" pad="P5"/>
+<contactref element="J1" pad="P3"/>
+<contactref element="J1" pad="P4"/>
+<contactref element="J1" pad="P1"/>
+<contactref element="J1" pad="P2"/>
 <wire x1="-57.15" y1="-202" x2="-57.15" y2="-197" width="0" layer="19" extent="1-1"/>
 <wire x1="-57.15" y1="-207" x2="-57.15" y2="-202" width="0" layer="19" extent="1-1"/>
@@
 <wire x1="50.02323125" y1="30.762303125" x2="51.091784375" y2="30.09655625" width="0" layer="19" extent="1-1"/>
 <wire x1="48.688509375" y1="26.13449375" x2="49" y2="30" width="0" layer="19" extent="1-1"/>
+<wire x1="19.34" y1="50.52" x2="14" y2="46.57260625" width="0" layer="19" extent="16-16"/>
+<wire x1="27.12" y1="50.52" x2="19.34" y2="50.52" width="0" layer="19" extent="16-16"/>
+<wire x1="31.425" y1="51.315" x2="27.12" y2="50.52" width="0" layer="19" extent="16-16"/>
+<wire x1="26.94" y1="55.05" x2="27.12" y2="50.52" width="0" layer="19" extent="1-16"/>
+<wire x1="31.525" y1="62.645" x2="28" y2="55" width="0" layer="19" extent="16-16"/>
+<wire x1="38.67384375" y1="57.42170625" x2="31.525" y2="62.645" width="0" layer="19" extent="16-16"/>
+<wire x1="39.797259375" y1="58.01401875" x2="38.67384375" y2="57.42170625" width="0" layer="19" extent="1-1"/>
 <wire x1="42" y1="15" x2="35.533203125" y2="21.4557" width="0" layer="19" extent="1-1"/>
 <wire x1="39" y1="9" x2="42" y2="15" width="0" layer="19" extent="1-1"/>
 <wire x1="34.825" y1="9.24" x2="37.775" y2="9.24" width="0" layer="19" extent="1-1"/>
-<wire x1="28" y1="55" x2="28.4" y2="40.9" width="0" layer="19" extent="1-1"/>
 <wire x1="21.68" y1="63.275" x2="26.94" y2="55.05" width="0" layer="19" extent="1-16"/>
-<wire x1="38.67384375" y1="57.42170625" x2="28" y2="55" width="0" layer="19" extent="1-1"/>
-<wire x1="39.797259375" y1="58.01401875" x2="38.67384375" y2="57.42170625" width="0" layer="19" extent="1-1"/>
+<wire x1="17.135" y1="62.795" x2="21.68" y2="63.275" width="0" layer="19" extent="16-16"/>
 </signal>
 <signal name="!RESET">
@@
 <contactref element="U$1" pad="3"/>
 <contactref element="CR1" pad="2"/>
-<contactref element="J14" pad="1"/>
 <contactref element="J5" pad="6"/>
 <wire x1="-81.28" y1="-368.37" x2="-84.7979" y2="-381" width="0" layer="19" extent="1-1"/>
 <wire x1="-116.64" y1="-401.32" x2="-84.7979" y2="-381" width="0" layer="19" extent="1-1"/>
-<wire x1="11.05" y1="9.3" x2="-81.28" y2="-368.37" width="0" layer="19" extent="1-16"/>
 </signal>
 <signal name="+12V">
@@
 <contactref element="U$7" pad="P$1"/>
 <contactref element="CR1" pad="1"/>
-<contactref element="J14" pad="2"/>
 <contactref element="J5" pad="14"/>
 <wire x1="-116.64" y1="-407.82" x2="-85.6869" y2="-381" width="0" layer="19" extent="1-1"/>
 <wire x1="-77.47" y1="-340.36" x2="-85.6869" y2="-381" width="0" layer="19" extent="1-1"/>
 <wire x1="-54.578" y1="-283" x2="-77.47" y2="-340.36" width="0" layer="19" extent="1-1"/>
-<wire x1="13.55" y1="9.3" x2="-54.578" y2="-283" width="0" layer="19" extent="1-16"/>
 </signal>
 <signal name="VCCA">
@@
 <contactref element="J5" pad="10"/>
 </signal>
+<signal name="READY">
+<contactref element="U3" pad="14"/>
+<contactref element="U9" pad="9"/>
+<wire x1="17.19" y1="44.245" x2="-52.67" y2="-63" width="0" layer="19" extent="1-1"/>
+</signal>
 </signals>
 <mfgpreviewcolors>
@@
 </drawing>
 <compatibility>
-<note version="6.3" minversion="6.2.2" severity="warning">
-Since Version 6.2.2 text objects can contain more than one line,
-which will not be processed correctly with this version.
-</note>
 <note version="8.2" severity="warning">
 Since Version 8.2, EAGLE supports online libraries. The ids
