File: pcb/microfloat.brd (EAGLE design)
At the start: 76.2 x 60.3 mm, 156 parts, among them J1 503182-1852, J2 1054291110, J3 USB4105_REVA, J4 1054291110, J5 JTAG-MINI, J6 1909763-1, J7 1054291110, J8 1054291110, T100 MMBT3906, U1 TXB0104PWR, U100 TPS54308DDCT, U101 LTC4419CMSEPBF, U102 MAX13237EETE, U103 TPS54308DDCT, U104 TPS54308DDCT, U105 TPS54308DDCT, U2 ICM-42688-P, U3 ATSAMD51N20A-AUT, U4 NEO-M8N-0, U5 BME280, Y1 ABS25-32.768KHZ-6-1-T

Commit message: Pain
Connections:
- net IMU_INT: now also U3.58; no longer U3.70
- net UART_RX_CTD_A: now also U1.5; no longer U1.3
- net UART_RX_CTD_B: now also U1.10; no longer U1.12
- net UART_RX_M_A: now also U1.3; no longer U1.5
- net UART_RX_M_B: now also U1.12; no longer U1.10
- net UART_TX_CTD_A: now also U1.4; no longer U1.2
- net UART_TX_CTD_B: now also U1.11; no longer U1.13
- net UART_TX_M_A: now also U1.2; no longer U1.4
- net UART_TX_M_B: now also U1.13; no longer U1.11
Routing:
- net UART_TX_M_A: track 0.00 -> 18.8 mm, vias 0 -> 2
- net UART_RX_M_A: track 0.00 -> 18.4 mm, vias 0 -> 2
- net IMU_INT: track 0.00 -> 10.1 mm, vias 0 -> 1
- net ANT_SW: track 0.00 -> 9.82 mm
- net UART_RX_CTD_A: track 11.2 -> 9.87 mm
- net UART_TX_CTD_A: track 11.3 -> 9.96 mm
- net UART_TX_CTD_B: track 16.6 -> 17.6 mm
- net UART_RX_CTD_B: track 20.4 -> 21.0 mm

Commit message: Names are a thing
Parts:
- moved U$15 45.5 mm to (36.0, 21.0)
- moved U$8 2.00 mm to (-11.5, 20.8)
- flipped R1 to the bottom, turned to 0 degrees
- flipped R2 to the bottom
Routing:
- net UART_TX_M_B: track 0.00 -> 52.9 mm, vias 0 -> 1
- net UART_RX_M_B: track 0.00 -> 9.27 mm, vias 0 -> 1
- net +6V: track 12.6 -> 13.8 mm
- net RREF+: track 37.6 -> 38.1 mm, vias 2 -> 3
- net RSENSE+: track 40.8 -> 41.0 mm, vias 2 -> 3
Other:
- board text added: "Designed by: Asha Arvind"
- board text added: "ECE/ME 4723 Group sd21p05"

Commit message: More changes
Parts:
- removed R103: 68k, rcl:R0603
- removed R104: 43k, rcl:R0603
- removed U$100: SQ2348ES-T1_GE3, microfloat:SOT-23-3
- removed U$101: GSOT04-E3-08, microfloat:SOT-23-3
- removed U$12, U$13: TEST_POINT, microfloat:TEST_POINT
- removed U$15: (no value), RoboJackets-Aesthetics:ROBOBUZZ_0.6X
- added $$$$U$3, $$$$U$4, $$$$U$5, $$U$1: TEST_POINT, microfloat:TEST_POINT
- added $$U$3: LR62E, microfloat:LR62E
- added R34: 1k', rcl:R0603
- added R35: 649, rcl:R0603
- $$U$10: value TEST_POINT -> SQ2348ES-T1_GE3; device microfloat:TEST_POINT -> microfloat:SOT-23-3
- $$U$11: value TEST_POINT -> GSOT04-E3-08; device microfloat:TEST_POINT -> microfloat:SOT-23-3
- C5: value 22uF -> 100uF; device rcl:C0805 -> rcl:E3,5-8
- C6: value 100uF -> 22uF; device rcl:E3,5-8 -> rcl:C0805
- J6: value 1909763-1 -> 1054291110; device microfloat:TE_1909763-1 -> microfloat:CON_1054291110_MOL
- J8: value 1054291110 -> 1909763-1; device microfloat:CON_1054291110_MOL -> microfloat:TE_1909763-1
- R1: value 649 -> 68k
- R2: value 1k' -> 43k
- U$6: value LR62E -> (none); device microfloat:LR62E -> RoboJackets-Aesthetics:ROBOBUZZ_0.6X
- moved $$U$4 66.6 mm to (-11.5, 20.8)
- moved R1 52.9 mm to (48.0, 23.5), turned to 180 degrees
- moved R2 49.8 mm to (45.0, 23.5), turned to 180 degrees
- moved $$U$10 45.6 mm to (6.00, 45.0), flipped to the bottom
- moved U$9 44.5 mm to (29.5, 45.2)
- moved U$8 27.4 mm to (6.50, 41.5)
- moved J6 22.6 mm to (21.8, 62.0), turned to 0 degrees
- moved J8 22.6 mm to (43.5, 56.0), turned to 270 degrees
- moved $$U$5 16.1 mm to (-12.3, 30.0)
- moved U$6 14.8 mm to (36.0, 21.0), turned to 0 degrees
- moved $$U$11 11.4 mm to (13.0, 47.0), flipped to the bottom, turned to 180 degrees
- moved C5 7.36 mm to (-4.25, 47.2), turned to 0 degrees
- moved C6 7.36 mm to (3.00, 46.0), turned to 180 degrees
- renumbered $$U$14 to $$U$7, $$U$16 to $$$$U$8, $$U$17 to $$$$U$6, $$U$18 to $$$$U$9, C100 to C16, C101 to C17, C102 to C13, C103 to C14, C104 to C9, C105 to C18, C106 to C15, C107 to C10, C108 to C19, C109 to C11, C110 to C12, C111 to C26, C112 to C27, C113 to C28, C114 to C32, C115 to C36, C116 to C24, C117 to C33, C118 to C22, C119 to C25, C120 to C30, C121 to C34, C122 to C37, C123 to C39, C124 to C21, C125 to C20, C126 to C31, C127 to C35, C128 to C38, C129 to C40, C130 to C41, C131 to C29, C132 to C23, C133 to C47, C134 to C46, C135 to C51, C136 to C52, C137 to C48, C138 to C54, C139 to C42, C140 to C49, C141 to C53, C142 to C55, C143 to C56, C144 to C50, C145 to C43, C146 to C44, C147 to C45, C148 to C58, C149 to C64, C150 to C57, C151 to C60, C152 to C62, C153 to C63, C154 to C59, C155 to C61, C156 to C65, CR100 to CR1, F100 to F1, F101 to F2, F102 to F3, F103 to F4, F104 to F5, F105 to F6, L100 to L2, L101 to L4, L102 to L3, L103 to L5, L104 to L6, R100 to R3, R101 to R4, R102 to R5, R105 to R13, R106 to R14, R107 to R15, R108 to R16, R109 to R17, R110 to R12, R111 to R6, R112 to R11, R113 to R8, R114 to R7, R115 to R9, R116 to R10, R117 to R18, R118 to R21, R119 to R22, R120 to R23, R121 to R24, R122 to R19, R123 to R20, R124 to R25, R125 to R26, R126 to R30, R127 to R31, R128 to R29, R129 to R32, R130 to R27, R131 to R33, R132 to R28, T100 to T1, U100 to U6, U101 to U8, U102 to U9, U103 to U7, U104 to U10, U105 to U11
Connections:
- net !SX-NRESET: now also $$U$3.P$2; no longer U$6.P$2
- net +12V: now also U$8.P$1; no longer U$12.P$1
- net +3V3: now also $$U$3.P$5, R34.2, R35.2; no longer R1.2, R2.2, U$6.P$5
- net +5V: now also $$U$5.P$1; no longer U$9.P$1
- net +6V: now also $$U$4.P$1; no longer U$8.P$1
- net ANT_SW: now also $$U$3.P$1; no longer U$6.P$1
- net CS_RAD: now also $$U$3.P$9; no longer U$6.P$9
- net GND: now also $$U$1.P$1, $$U$10.2, $$U$11.3, $$U$3.P$10, C5.-, C6.2, J6.11, J6.12, J6.8, J6.9, J8.2, J8.3, R2.1, U$9.P$1; no longer $$U$5.P$1, C5.2, C6.-, J6.2, J6.3, J8.11, J8.12, J8.8, J8.9, R104.1, U$100.2, U$101.3, U$13.P$1, U$6.P$10
- net GPS_ANT: now also J8.1; no longer J6.1
- net MISO_2: now also $$U$3.P$8; no longer U$6.P$8
- net MOSI_2: now also $$U$3.P$7; no longer U$6.P$7
- net N$17: now also C6.1; no longer C5.1
- net N$21: now also R1.2; no longer R103.2
- net N$22: now also R1.1, R2.2; no longer R103.1, R104.2
- net N$24: now also $$U$10.1; no longer U$100.1
- net PROBE: now also J6.10, J6.5; no longer J8.10, J8.5
- net RAD_BUSY: now also $$U$3.P$3; no longer U$6.P$3
- net RREF+: now also J6.3, R34.1; no longer J8.3, R2.1
- net RSENSE+: now also J6.4, R35.1; no longer J8.4, R1.1
- net SCLK_2: now also $$U$3.P$6; no longer U$6.P$6
- net SOLENOID: now also $$U$11.1; no longer U$101.1
- net SOL_TRIG: now also $$U$10.3; no longer U$100.3
- net VBATT: now also $$$$U$5.P$1, C5.+; no longer $$U$11.P$1, C6.+
- net VBATT_5V: now also $$$$U$4.P$1; no longer $$U$10.P$1
- net VBUS: now also $$$$U$3.P$1; no longer $$U$4.P$1
- net VIN: now also J6.1; no longer J8.1

Commit message: no airwires, clearance issues, dimensions, wire stubs
Parts:
- removed U$6: (no value), RoboJackets-Aesthetics:ROBOBUZZ_0.6X
- moved L1 1.13 mm to (19.8, 43.3)
- moved $$U$4 0.51 mm to (-11.6, 21.3)
- moved C9 0.50 mm to (45.0, 16.5)
- moved C10 0.40 mm to (45.0, 18.6)
- moved C11 0.30 mm to (45.0, 20.7)
Routing:
- net UART_RX_M_B: track 9.27 -> 68.3 mm, vias 1 -> 9
- net ANT_SW: track 9.82 -> 57.0 mm, vias 0 -> 5
- net CS_PHT: track 0.00 -> 42.8 mm, vias 0 -> 6
- net RAD_BUSY: track 0.00 -> 37.2 mm, vias 0 -> 4
- net MOSI_1: track 15.2 -> 47.1 mm, vias 0 -> 6
- net MISO_1: track 18.6 -> 49.8 mm, vias 0 -> 4
- net CS_GPS: track 0.00 -> 31.2 mm, vias 0 -> 2
- net SCLK_1: track 17.5 -> 47.9 mm, vias 2 -> 7
- net UART_TX_M_B: track 52.9 -> 69.9 mm, vias 1 -> 5
- net IMU_INT: track 10.1 -> 14.1 mm, vias 1 -> 2
- net GND: track 187.9 -> 190.8 mm, vias 132 -> 131
- net VBATT: track 135.8 -> 138.3 mm
- net +3V3: track 74.9 -> 77.0 mm
- net T_OUT: track 17.4 -> 19.3 mm
- net TX_READY: track 27.5 -> 29.4 mm
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
Commit message: BEEG Capacitor
Parts:
- removed C42, C64: 33uF, rcl:C1206
- added C66, C67: KCM55TR7YA336MH01L, microfloat:CAPC6153X500N
- moved $$U$4 5.50 mm to (-12.2, 26.8)
- moved C6 1.00 mm to (3.00, 45.0)
- moved C7 1.00 mm to (3.00, 47.0)
- flipped BT1 to the bottom
Connections:
- net GND: now also C66.1, C67.1; no longer C42.2, C64.2
- net VBATT: now also C66.2, C67.2; no longer C42.1, C64.1
Routing:
- net +6V: track 13.4 -> 15.0 mm
- net N$17: track 21.2 -> 22.8 mm
- net GND: track 190.8 -> 191.6 mm, vias 131 -> 130
- net VBATT: track 138.3 -> 138.8 mm
Other:
- board text removed: "Designed by: Asha Arvind"

Commit message: Changes I think
Parts:
- L2: value 13uH -> 10uH
- L3: value 12uH -> 10uH
- L6: value 6.471uH -> 3.9uH
- moved C67 41.6 mm to (41.9, 31.7), turned to 90 degrees
Routing:
- net VBATT: track 138.8 -> 147.7 mm, vias 6 -> 7
- net GND: track 191.6 -> 195.8 mm, vias 130 -> 131
- net D_N: track 36.3 -> 37.1 mm

Commit message: Last inductor to fix
Parts:
- removed $$$$U$9: (no value), HyTechAesthetics:LOGO_GT_0.25"
- removed $$U$10: SQ2348ES-T1_GE3, microfloat:SOT-23-3
- removed $$U$3: LR62E, microfloat:LR62E
- removed $$U$7, U$7, U$8: TEST_POINT, microfloat:TEST_POINT
- removed C66, C67: KCM55TR7YA336MH01L, microfloat:CAPC6153X500N
- added $$$$$$U$1, $$$$$$U$2, $$$$$$U$3, $$$$U$2: TEST_POINT, microfloat:TEST_POINT
- added $$$$U$1: (no value), HyTechAesthetics:LOGO_GT_0.25"
- added C42: 0.1uF, rcl:C0603
- added C64: 100nF, rcl:C0603
- added U12, U13: TPS54308DDCT, microfloat:SOT95P280X110-6N
- $$U$4: value TEST_POINT -> (none); device microfloat:TEST_POINT -> RoboJackets-Aesthetics:ROBOBUZZ_0.4X
- C10: value 10 uF -> 10uF; device rcl:C0603 -> rcl:E2,5-5
- C11: value 0.1 uF -> 10uF; device rcl:C0603 -> rcl:C0805
- C12: device rcl:C0603 -> rcl:C0805
- C15: value 100nF -> 1.0 uF
- C16, C44: value 10uF -> 22uF
- C17: value 10uF -> 100nF; device rcl:C0805 -> rcl:C0603
- C18: value 22uF -> 10 uF; device rcl:C0805 -> rcl:C0603
- C2: value 0.1uF -> KCM55TR7YA336MH01L; device rcl:C0603 -> microfloat:CAPC6153X500N
- C20: value 10uF -> 0.1 uF
- C21: value 100nF -> 10uF
- C22: value 10uF -> 2.2 uF
- C23: value 0.1uF -> 0.1 uF
- C24: value 0.1uF -> 0.01 uF
- C25: value 0.1uF -> 10uF; device rcl:C0603 -> rcl:C0805
- C26: value 2.2 uF -> 0.1uF
- C27: value 0.1 uF -> 0.1uF
- C28: value 0.01 uF -> 10uF; device rcl:C0603 -> rcl:C0805
- C29, C36: value 0.1uF -> 10uF
- C32, C33, C55: value 10uF -> 0.1uF; device rcl:C0805 -> rcl:C0603
- C35: value 0.1uF -> 100nF
- C45: value 1.0uF -> 22uF
- C46: value 22uF -> 0.1uF
- C47: value 22uF -> 4.7uF
- C5: value 100uF -> 0.1uF; device rcl:E3,5-8 -> rcl:C0603
- C52: value 4.7uF -> 10uF; device rcl:C0603 -> rcl:C0805
- C53: value 0.1uF -> 8.2 pF
- C56: value 8.2 pF -> 10uF
- C57: value 0.1 uF -> 1.0uF
- C61: value 100nF -> 22uF
- C63: value 22uF -> 0.1 uF
- C8: value 10uF -> 100uF; device rcl:E2,5-5 -> rcl:E3,5-8
- C9: value 1.0 uF -> KCM55TR7YA336MH01L; device rcl:C0603 -> microfloat:CAPC6153X500N
- J6: value 1054291110 -> 1909763-1; device microfloat:CON_1054291110_MOL -> microfloat:TE_1909763-1
- J8: value 1909763-1 -> 1054291110; device microfloat:TE_1909763-1 -> microfloat:CON_1054291110_MOL
- L1, L2, L3: device RoboJackets-Inductors:0805 -> microfloat:78438357100
- L5, L6: device RoboJackets-Inductors:0805 -> microfloat:SRR3818A-3R9Y
- R1: value 68k -> 100k
- R11: value 910k -> 82k
- R12: value 82k -> 5.1k
- R13: value 100k -> 910k
- R14: value 10k -> 390k
- R15: value 10k -> 5.1k
- R16: value 100k -> 13.7k
- R19: value 100k -> 150k
- R2: value 43k -> 100k
- R20: value 10 -> 100k
- R21: value 150k -> 100k
- R22: value 100k -> 560k
- R24: value 560k -> 10
- R27: value 100k -> 1k
- R28: value 22k -> 1k
- R3: value 100k -> 11k
- R30, R31: value 1k -> 100k
- R32: value 100k -> 5.23k
- R33: value 5.23k -> 22k
- R4: value 100k -> 68k
- R5: value 11k -> 43k
- R6: value 5.1k -> 100k
- R7: value 5.1k -> 10k
- R8: value 390k -> 10k
- R9: value 13.7k -> 100k
- U11: value TPS54308DDCT -> SQ2348ES-T1_GE3; device microfloat:SOT95P280X110-6N -> microfloat:SOT-23-3
- U2: value ICM-42688-P -> LR62E; device microfloat:PQFN50P300X250X97-14N -> microfloat:LR62E
- U3: value ATSAMD51N20A-AUT -> ICM-42688-P; device microfloat:QFP50P1600X1600X120-100N -> microfloat:PQFN50P300X250X97-14N
- U4: value NEO-M8N-0 -> ATSAMD51N20A-AUT; device microfloat:XCVR_NEO-M8N-0 -> microfloat:QFP50P1600X1600X120-100N
- U5: value BME280 -> NEO-M8N-0; device microfloat:PSON65P250X250X100-8N -> microfloat:XCVR_NEO-M8N-0
- U6: value TPS54308DDCT -> BME280; device microfloat:SOT95P280X110-6N -> microfloat:PSON65P250X250X100-8N
- moved $$$$U$3 68.5 mm to (-12.2, 26.8)
- moved U6 63.4 mm to (50.2, 50.8), flipped to the top, turned to 270 degrees
- moved $$$$U$4 63.0 mm to (-12.3, 30.0)
- moved $$U$4 61.3 mm to (49.0, 24.0)
- moved C10 58.4 mm to (-1.50, 54.0), flipped to the top, turned to 0 degrees
- moved R4 54.0 mm to (48.0, 23.5), turned to 180 degrees
- moved C9 53.8 mm to (5.00, 52.5), flipped to the top, turned to 90 degrees
- moved U7 53.5 mm to (-4.00, 18.0), turned to 90 degrees
- moved C18 53.0 mm to (45.0, 18.6), turned to 180 degrees
- moved R15 52.7 mm to (57.5, 30.0), turned to 0 degrees
- moved R2 51.0 mm to (-6.00, 21.2), turned to 0 degrees
- moved R5 51.0 mm to (45.0, 23.5)
- moved R7 50.7 mm to (7.00, 25.0), turned to 90 degrees
- moved C11 49.5 mm to (-4.00, 13.5), turned to 270 degrees
- moved R6 48.6 mm to (9.00, 25.0), turned to 90 degrees
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- renumbered $$$$U$6 to $$$$$$U$5, $$$$U$8 to $$$$$$U$4, $$U$11 to D1, U$9 to U$6
Connections:
- net !RESET: now also U4.88; no longer U3.88
- net !RESET_N: now also U4.72, U5.8; no longer U3.72, U4.8
- net !SX-NRESET: now also U2.P$2, U4.68; no longer $$U$3.P$2, U3.68
- net +12V: now also $$U$5.P$1; no longer U$8.P$1
- net +3V3: now also $$$$U$5.P$1, C15.1, C18.1, C20.1, C22.1, C23.1, C24.1, C25.1, C42.1, C46.1, C5.1, C55.1, C56.1, C63.1, R1.1, R10.2, R6.2, R7.2, R8.2, R9.2, U2.P$5, U3.5, U3.8, U4.25, U4.30, U4.39, U4.51, U4.63, U4.77, U4.92, U5.23, U6.6, U6.8; no longer $$U$3.P$5, $$U$7.P$1, C10.1, C11.1, C27.1, C29.1, C3.1, C30.1, C35.1, C36.1, C43.1, C44.1, C45.1, C51.1, C9.1, R13.2, R14.2, R15.2, R16.2, R17.2, R3.1, U2.5, U2.8, U3.25, U3.30, U3.39, U3.51, U3.63, U3.77, U3.92, U4.23, U5.6, U5.8
- net +5V: now also $$$$U$4.P$1, C21.1, U12.3; no longer $$U$5.P$1, C12.1, U10.3
- net +6V: now also $$$$U$3.P$1; no longer $$U$4.P$1
- net ANT_SW: now also U2.P$1, U4.69; no longer $$U$3.P$1, U3.69
- net BATT_MEASURE: now also R21.2, R22.1, U4.15; no longer R23.2, R24.1, U3.15
- net CO2_IN: now also R20.2; no longer R22.2
- net CO2_OUT: now also R19.2, R20.1, U4.13; no longer R21.2, R22.1, U3.13
- net CS_GPS: now also U4.48, U5.18; no longer U3.48, U4.18
- net CS_IMU: now also U3.12, U4.55; no longer U2.12, U3.55
- net CS_PHT: now also U4.83, U6.2; no longer U3.83, U5.2
- net CS_RAD: now also U2.P$9, U4.49; no longer $$U$3.P$9, U3.49
- net D_N: now also U4.74; no longer U3.74
- net D_P: now also U4.75; no longer U3.75
- net GND: now also $$$$U$2.P$1, C10.-, C15.2, C2.1, C21.2, C23.2, C24.2, C25.2, C42.2, C5.2, C61.2, C9.1, J6.2, J6.3, J8.11, J8.12, J8.8, J8.9, R11.1, R12.2, R15.1, R16.1, R3.1, R32.1, U11.2, U12.1, U13.1, U2.P$10, U3.10, U3.2, U3.3, U3.6, U3.7, U4.11, U4.31, U4.38, U4.50, U4.62, U4.76, U4.90, U5.10, U5.12, U5.13, U5.2, U5.24, U6.7; no longer $$U$10.2, $$U$3.P$10, C10.2, C17.2, C2.2, C27.2, C30.2, C35.2, C43.2, C5.-, C66.1, C67.1, C9.2, J6.11, J6.12, J6.8, J6.9, J8.2, J8.3, R12.1, R2.1, R31.1, R6.2, R7.1, R9.1, U$3.P$1, U11.1, U2.10, U2.11, U2.2, U2.3, U2.6, U2.7, U3.24, U3.31, U3.38, U3.50, U3.62, U3.76, U3.90, U4.10, U4.12, U4.13, U4.2, U4.7, U5.1
- net GPS_ANT: now also J6.1, U5.11; no longer J8.1, U4.11
- net IMU_INT: now also U3.4, U4.58; no longer U2.4, U3.58
- net LEAK: now also R28.2, U4.36; no longer R31.2, U3.36
- net LNA_EN: now also U4.73, U5.14; no longer U3.73, U4.14
- net MISO_1: now also U4.82, U5.20, U6.5; no longer U3.82, U4.20, U5.5
- net MISO_2: now also U2.P$8, U3.1, U4.54; no longer $$U$3.P$8, U2.1, U3.54
- net MODEM_R_IN: now also U4.56; no longer U3.56
- net MODEM_T_IN: now also U4.57; no longer U3.57
- net MOSI_1: now also U4.80, U5.21, U6.3; no longer U3.80, U4.21, U5.3
- net MOSI_2: now also U2.P$7, U3.14, U4.52; no longer $$U$3.P$7, U2.14, U3.52
- net N$1: now also R1.2; no longer R3.2
- net N$10: now also C54.1; no longer C49.1
- net N$11: now also C35.1, U10.6; no longer C21.1, U7.6
- net N$12: now also C35.2, L1.2, U10.2; no longer C21.2, L3.1, U7.2
- net N$13: now also R16.2, R17.1, U10.4; no longer R10.1, R9.2, U7.4
- net N$14: now also C64.1, U12.6; no longer C61.1, U10.6
- net N$15: now also C64.2, U12.2; no longer C61.2, U10.2
- net N$16: now also R31.1, R33.2, U12.4; no longer R27.1, R28.2, U10.4
- net N$17: now also R30.2; no longer R32.2
- net N$18: now also C16.1, L3.1, R2.2; no longer C18.1, L2.2, R4.2
- net N$19: now also C44.1, C45.1, L1.1, R17.2; no longer C46.1, C47.1, L3.2, R10.2
- net N$2: now also C43.1; no longer C23.1
- net N$20: now also C61.1, R31.2; no longer C63.1, R27.2
- net N$21: now also R14.1, R4.2; no longer R1.2, R8.1
- net N$22: now also R4.1, R5.2; no longer R1.1, R2.2
- net N$23: now also R11.2, R13.1; no longer R11.1, R12.2
- net N$24: now also R24.1, U11.1; no longer $$U$10.1, R20.1
- net N$25: now also L2.2, U4.91; no longer L1.1, U3.91
- net N$26: now also C36.1, R14.2; no longer C20.1, R8.2
- net N$28: now also U$3.P$1; no longer U$7.P$1
- net N$3: now also R27.1; no longer R30.1
- net N$32: now also U5.22; no longer U4.22
- net N$35: now also U13.6; no longer U11.6
- net N$36: now also U13.2; no longer U11.2
- net N$37: now also R30.1, R32.2, U13.4; no longer R32.1, R33.2, U11.4
- net N$38: now also C17.1, U7.6; no longer C15.1, U6.6
- net N$39: now also C17.2, L3.2, U7.2; no longer C15.2, L2.1, U6.2
- net N$4: now also C43.2; no longer C23.2
- net N$40: now also R2.1, R3.2, U7.4; no longer R4.1, R5.2, U6.4
- net N$5: now also C27.1, C30.1; no longer C24.1, C25.1
- net N$6: now also C27.2, C30.2; no longer C24.2, C25.2
- net N$7: now also R15.2; no longer R7.2
- net N$8: now also C3.1; no longer C2.1
- net N$9: now also R12.1; no longer R6.1
- net PROBE: now also J8.10, J8.5, R27.2; no longer J6.10, J6.5, R30.2
- net RAD_BUSY: now also U2.P$3, U4.79; no longer $$U$3.P$3, U3.79
- net READY: now also U4.71; no longer U3.71
- net RREF+: now also J8.3, U4.97; no longer J6.3, U3.97
- net RSENSE+: now also J8.4, U4.99; no longer J6.4, U3.99
- net SCLK_1: now also U4.81, U5.19, U6.4; no longer U3.81, U4.19, U5.4
- net SCLK_2: now also U2.P$6, U3.13, U4.53; no longer $$U$3.P$6, U2.13, U3.53
- net SD_CD: now also R7.1, U4.19; no longer R14.1, U3.19
- net SD_CK: now also U4.33; no longer U3.33
- net SD_CMD: now also R8.1, U4.26; no longer R15.1, U3.26
- net SD_DATA0: now also R9.1, U4.27; no longer R16.1, U3.27
- net SD_DATA1: now also R10.1, U4.28; no longer R17.1, U3.28
- net SD_DATA2: now also R6.1, U4.29; no longer R13.1, U3.29
- net SOLENOID: now also R23.2, R24.2, U4.37; no longer R19.2, R20.2, U3.37
- net SOL_TRIG: now also U11.3; no longer $$U$10.3
- net SWCLK: now also U4.93; no longer U3.93
- net SWDIO: now also U4.94; no longer U3.94
- net TX_READY: now also U4.78, U5.4; no longer U3.78, U4.4
- net UART_RX_CTD_A: now also U4.34; no longer U3.34
- net UART_RX_M_A: now also U4.64; no longer U3.64
- net UART_RX_PH: now also U4.46; no longer U3.46
- net UART_TX_CTD_A: now also U4.35; no longer U3.35
- net UART_TX_M_A: now also U4.65; no longer U3.65
- net UART_TX_PH: now also U4.47; no longer U3.47
- net VBATT: now also $$$$$$U$3.P$1, C10.+, C11.1, C12.1, C2.2, C9.2, R22.2, U10.3, U13.3; no longer $$$$U$5.P$1, C16.1, C17.1, C5.+, C66.2, C67.2, R24.2, U11.3, U6.3
- net VBATT_5V: now also $$$$$$U$2.P$1, C29.1, R13.2; no longer $$$$U$4.P$1, C22.1, R11.2
- net VBUS: now also $$$$$$U$1.P$1; no longer $$$$U$3.P$1
- net VCCA: now also C49.1, C52.1, U4.12; no longer C54.1, C55.1, U3.12
- net VCC_CORE: now also C47.1, C51.1, L2.1, U4.89; no longer C52.1, C53.1, L1.2, U3.89
- net VIN: now also J8.1; no longer J6.1
- net XIN32: now also C53.1, U4.1; no longer C56.1, U3.1
- net XOUT32: now also U4.2; no longer U3.2
Routing:
- net GND: track 195.8 -> 210.3 mm, vias 131 -> 127
- net N$19: track 11.5 -> 17.9 mm, vias 0 -> 1
- net VCC_CORE: track 8.95 -> 14.8 mm
- net +5V: track 125.8 -> 129.1 mm, vias 3 -> 4
- net UART_RX_M_B: track 68.3 -> 70.0 mm, vias 9 -> 8
- net VBATT_5V: track 19.5 -> 21.0 mm
- net N$15: track 6.00 -> 7.29 mm
- net N$25: track 3.46 -> 4.66 mm, vias 0 -> 1
- net SWCLK: track 46.0 -> 44.9 mm
- net N$18: track 15.7 -> 16.8 mm
- net N$12: track 11.2 -> 10.1 mm, vias 0 -> 1
- net SWDIO: track 47.5 -> 46.5 mm
- net SCLK_1: track 47.9 -> 47.1 mm
- net N$39: track 6.03 -> 6.85 mm
Other:
- board text added: "Designed by: Asha B Arvind S"
- board text added: "MicroFloats!"

Commit message: One last DRC error
Parts:
- moved L6 4.92 mm to (-3.90, 50.6)
Routing:
- net N$36: track 8.31 -> 19.1 mm
- net N$17: track 22.8 -> 28.8 mm
- net VIN: track 41.8 -> 36.7 mm, vias 3 -> 4
- net VBATT: track 147.5 -> 148.3 mm
