File: pcb/microfloat.sch (EAGLE design)
At the start: 152 parts, among them J1 503182-1852, J2 USB4105_REVA, J3 1054291110, J4 1054291110, J6 JTAG-MINI, J7 1054291110, J8 1054291110, J9 1909763-1, T1 MMBT3906, U1 BME280, U12 TPS54308DDCT, U13 TPS54308DDCT, U2 ICM-42688-P, U3 MAX13237EETE, U4 NEO-M8N-0, U5 TXB0104PWR, U6 LTC4419CMSEPBF, U7 TPS54308DDCT, U8 TPS54308DDCT, U9 ATSAMD51N20A-AUT, Y1 ABS25-32.768KHZ-6-1-T

Commit message: Pain
Parts:
- C17, C53: device rcl:C-USC0603 -> rcl:C-USC1206
- C21, C37, C52, C55, C57, C59, C60: device rcl:C-USC0603 -> rcl:C-USC0805
Changed lines of the file:
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@@
 <part name="FRAME3" library="frames" library_urn="urn:adsk.eagle:library:229" deviceset="FRAME_B_L" device=""/>
 <part name="U12" library="microfloat" deviceset="TPS54308DDCT" device=""/>
-<part name="C53" library="rcl" library_urn="urn:adsk.eagle:library:334" deviceset="C-US" device="C0603" package3d_urn="urn:adsk.eagle:package:23616/2" value="33uF">
+<part name="C53" library="rcl" library_urn="urn:adsk.eagle:library:334" deviceset="C-US" device="C1206" package3d_urn="urn:adsk.eagle:package:23618/2" value="33uF">
 <spice>
 <pinmapping spiceprefix="C">
@@
 <part name="GND53" library="supply1" library_urn="urn:adsk.eagle:library:371" deviceset="GND" device=""/>
 <part name="U13" library="microfloat" deviceset="TPS54308DDCT" device=""/>
-<part name="C57" library="rcl" library_urn="urn:adsk.eagle:library:334" deviceset="C-US" device="C0603" package3d_urn="urn:adsk.eagle:package:23616/2" value="10uF">
+<part name="C57" library="rcl" library_urn="urn:adsk.eagle:library:334" deviceset="C-US" device="C0805" package3d_urn="urn:adsk.eagle:package:23617/2" value="10uF">
 <spice>
 <pinmapping spiceprefix="C">
@@
 <attribute name="TOLERANCE" value="10%"/>
 </part>
-<part name="C59" library="rcl" library_urn="urn:adsk.eagle:library:334" deviceset="C-US" device="C0603" package3d_urn="urn:adsk.eagle:package:23616/2" value="22uF">
+<part name="C59" library="rcl" library_urn="urn:adsk.eagle:library:334" deviceset="C-US" device="C0805" package3d_urn="urn:adsk.eagle:package:23617/2" value="22uF">
 <spice>
 <pinmapping spiceprefix="C">
@@
 <part name="GND55" library="supply1" library_urn="urn:adsk.eagle:library:371" deviceset="GND" device=""/>
 <part name="U$23" library="microfloat" deviceset="VBATT" device=""/>
-<part name="C60" library="rcl" library_urn="urn:adsk.eagle:library:334" deviceset="C-US" device="C0603" package3d_urn="urn:adsk.eagle:package:23616/2" value="22uF">
+<part name="C60" library="rcl" library_urn="urn:adsk.eagle:library:334" deviceset="C-US" device="C0805" package3d_urn="urn:adsk.eagle:package:23617/2" value="22uF">
 <spice>
 <pinmapping spiceprefix="C">
@@
 <part name="GND27" library="supply1" library_urn="urn:adsk.eagle:library:371" deviceset="GND" device=""/>
 <part name="U7" library="microfloat" deviceset="TPS54308DDCT" device=""/>
-<part name="C17" library="rcl" library_urn="urn:adsk.eagle:library:334" deviceset="C-US" device="C0603" package3d_urn="urn:adsk.eagle:package:23616/2" value="33uF">
+<part name="C17" library="rcl" library_urn="urn:adsk.eagle:library:334" deviceset="C-US" device="C1206" package3d_urn="urn:adsk.eagle:package:23618/2" value="33uF">
 <spice>
 <pinmapping spiceprefix="C">
@@
 </part>
 <part name="GND30" library="supply1" library_urn="urn:adsk.eagle:library:371" deviceset="GND" device=""/>
-<part name="C21" library="rcl" library_urn="urn:adsk.eagle:library:334" deviceset="C-US" device="C0603" package3d_urn="urn:adsk.eagle:package:23616/2" value="10uF">
+<part name="C21" library="rcl" library_urn="urn:adsk.eagle:library:334" deviceset="C-US" device="C0805" package3d_urn="urn:adsk.eagle:package:23617/2" value="10uF">
 <spice>
 <pinmapping spiceprefix="C">
@@
 <attribute name="VOLTAGE" value="10V"/>
 </part>
-<part name="C37" library="rcl" library_urn="urn:adsk.eagle:library:334" deviceset="C-US" device="C0603" package3d_urn="urn:adsk.eagle:package:23616/2" value="10uF">
+<part name="C37" library="rcl" library_urn="urn:adsk.eagle:library:334" deviceset="C-US" device="C0805" package3d_urn="urn:adsk.eagle:package:23617/2" value="10uF">
 <spice>
 <pinmapping spiceprefix="C">
@@
 <attribute name="VOLTAGE" value="10V"/>
 </part>
-<part name="C52" library="rcl" library_urn="urn:adsk.eagle:library:334" deviceset="C-US" device="C0603" package3d_urn="urn:adsk.eagle:package:23616/2" value="22uF">
+<part name="C52" library="rcl" library_urn="urn:adsk.eagle:library:334" deviceset="C-US" device="C0805" package3d_urn="urn:adsk.eagle:package:23617/2" value="22uF">
 <spice>
 <pinmapping spiceprefix="C">
@@
 <attribute name="VOLTAGE" value="16V"/>
 </part>
-<part name="C55" library="rcl" library_urn="urn:adsk.eagle:library:334" deviceset="C-US" device="C0603" package3d_urn="urn:adsk.eagle:package:23616/2" value="22uF">
-<spice>
-<pinmapping spiceprefix="C">
+<part name="C55" library="rcl" library_urn="urn:adsk.eagle:library:334" deviceset="C-US" device="C0805" package3d_urn="urn:adsk.eagle:package:23617/2" value="22uF">
+<spice>
+<pinmapping spiceprefix="C">

Commit message: More pain
Parts:
- R25: value 652 -> 649
Connections:
- removed net !RESET!: R35.2
- removed net N$30: J8.11
- removed net N$31: J7.11
- net !RESET: now also R35.2
- net GND: now also J7.11, J8.11
Changed lines of the file:
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@@
 <part name="GND42" library="supply1" library_urn="urn:adsk.eagle:library:371" deviceset="GND" device=""/>
 <part name="+3V14" library="supply1" library_urn="urn:adsk.eagle:library:371" deviceset="+3V3" device=""/>
-<part name="R25" library="rcl" library_urn="urn:adsk.eagle:library:334" deviceset="R-US_" device="R0603" package3d_urn="urn:adsk.eagle:package:23555/3" value="652">
+<part name="R25" library="rcl" library_urn="urn:adsk.eagle:library:334" deviceset="R-US_" device="R0603" package3d_urn="urn:adsk.eagle:package:23555/3" value="649">
 <spice>
 <pinmapping spiceprefix="R">
@@
 <pinref part="J6" gate="G$1" pin="!RST"/>
 </segment>
+<segment>
+<pinref part="R35" gate="G$1" pin="2"/>
+<wire x1="182.88" y1="254" x2="180.34" y2="254" width="0.1524" layer="91"/>
+<label x="180.34" y="254" size="1.27" layer="95" rot="R180" xref="yes"/>
+</segment>
 </net>
 <net name="+3V3" class="0">
@@
 </segment>
 </net>
-<net name="!RESET!" class="0">
-<segment>
-<pinref part="R35" gate="G$1" pin="2"/>
-<wire x1="182.88" y1="254" x2="180.34" y2="254" width="0.1524" layer="91"/>
-<label x="180.34" y="254" size="1.27" layer="95" rot="R180" xref="yes"/>
-</segment>
-</net>
 <net name="TX_READY" class="0">
 <segment>
@@
 <segment>
 <pinref part="GND21" gate="1" pin="GND"/>
-<wire x1="363.22" y1="54.5338" x2="363.22" y2="53.34" width="0.1524" layer="91"/>
 <pinref part="J8" gate="A" pin="12"/>
 <wire x1="363.22" y1="53.34" x2="363.22" y2="50.8" width="0.1524" layer="91"/>
+<pinref part="J8" gate="A" pin="11"/>
+<wire x1="363.22" y1="55.88" x2="363.22" y2="53.34" width="0.1524" layer="91"/>
 <junction x="363.22" y="53.34"/>
 </segment>
 <segment>
 <pinref part="GND59" gate="1" pin="GND"/>
-<wire x1="398.78" y1="54.5338" x2="398.78" y2="53.34" width="0.1524" layer="91"/>
 <pinref part="J7" gate="A" pin="12"/>
 <wire x1="398.78" y1="53.34" x2="398.78" y2="50.8" width="0.1524" layer="91"/>
+<pinref part="J7" gate="A" pin="11"/>
+<wire x1="398.78" y1="55.88" x2="398.78" y2="53.34" width="0.1524" layer="91"/>
 <junction x="398.78" y="53.34"/>
 </segment>
@@
 </segment>
 </net>
-<net name="N$30" class="0">
-<segment>
-<wire x1="363.22" y1="55.88" x2="363.22" y2="54.6862" width="0.1524" layer="91"/>
-<pinref part="J8" gate="A" pin="11"/>
-</segment>
-</net>
-<net name="N$31" class="0">
-<segment>
-<wire x1="398.78" y1="55.88" x2="398.78" y2="54.6862" width="0.1524" layer="91"/>
-<pinref part="J7" gate="A" pin="11"/>
-</segment>
-</net>
