File: pcb/microfloat.sch (EAGLE design)
At the start: 152 parts, among them J1 503182-1852, J2 USB4105_REVA, J3 1054291110, J4 1054291110, J6 JTAG-MINI, J7 1054291110, J8 1054291110, J9 1909763-1, T1 MMBT3906, U1 BME280, U12 TPS54308DDCT, U13 TPS54308DDCT, U2 ICM-42688-P, U3 MAX13237EETE, U4 NEO-M8N-0, U5 TXB0104PWR, U6 LTC4419CMSEPBF, U7 TPS54308DDCT, U8 TPS54308DDCT, U9 ATSAMD51N20A-AUT, Y1 ABS25-32.768KHZ-6-1-T

Commit message: So much pain
Parts:
- added C11: 10 uF, rcl:C-USC0603
- added C8: 0.1 uF, rcl:C-USC0603
Connections:
- removed net N$27: C41.+, C42.+, F6.1
- new net VIN: F6.2
- net +3V3: now also C11.1, C8.1
- net GND: now also C11.2, C8.2
- net VBATT: now also C41.+, C42.+, F6.1; no longer F6.2
Other:
- moved on the sheet: C40, U$3

Commit message: Routing is hell
Parts:
- added U$35: TEST_POINT, microfloat:TEST_POINT
Connections:
- removed net RREF-: J8.7
- removed net RSENSE-: J8.8
- net GND: now also J8.8, J8.9
- net PROBE: now also J8.10, J8.5; no longer J8.4, J8.9
- net READY: now also U9.PA21; no longer U9.PB04
- net RREF+: now also J8.3; no longer J8.2
- net RSENSE+: now also J8.4; no longer J8.3
- net UART_RX_PH: now also J4.2; no longer J4.1
- net UART_TX_PH: now also J4.1; no longer J4.2
- net VBATT: now also U$35.P$1
- net VIN: now also J8.1
Changed lines of the file:
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@@
 <attribute name="TOLERANCE" value="0.1%"/>
 </part>
-<part name="GND40" library="supply1" library_urn="urn:adsk.eagle:library:371" deviceset="GND" device=""/>
 <part name="+3V17" library="supply1" library_urn="urn:adsk.eagle:library:371" deviceset="+3V3" device=""/>
 <part name="R26" library="rcl" library_urn="urn:adsk.eagle:library:334" deviceset="R-US_" device="R0603" package3d_urn="urn:adsk.eagle:package:23555/3" value="1k'">
@@
 <attribute name="TOLERANCE" value="0.1%"/>
 </part>
-<part name="GND44" library="supply1" library_urn="urn:adsk.eagle:library:371" deviceset="GND" device=""/>
 <part name="U9" library="microfloat" deviceset="ATSAMD51N20A-AUT" device=""/>
 <part name="FRAME3" library="frames" library_urn="urn:adsk.eagle:library:229" deviceset="FRAME_B_L" device=""/>
@@
 <part name="U$18" library="microfloat" deviceset="VIN" device=""/>
 <part name="U$30" library="microfloat" deviceset="VBATT" device=""/>
+<part name="U$34" library="microfloat" deviceset="VIN" device=""/>
+<part name="GND40" library="supply1" library_urn="urn:adsk.eagle:library:371" deviceset="GND" device=""/>
+<part name="U$35" library="microfloat" deviceset="TEST_POINT" device=""/>
 </parts>
 <sheets>
@@
 </segment>
 </net>
-<net name="READY" class="0">
-<segment>
-<pinref part="U9" gate="G$1" pin="PB04"/>
-<wire x1="66.04" y1="147.32" x2="63.5" y2="147.32" width="0.1524" layer="91"/>
-<label x="63.5" y="147.32" size="1.27" layer="95" rot="R180" xref="yes"/>
-</segment>
-</net>
 <net name="N$25" class="0">
 <segment>
@@
 </segment>
 </net>
+<net name="READY" class="0">
+<segment>
+<wire x1="66.04" y1="180.34" x2="63.5" y2="180.34" width="0.1524" layer="91"/>
+<label x="63.5" y="180.34" size="1.27" layer="95" rot="R180" xref="yes"/>
+<pinref part="U9" gate="G$1" pin="PA21"/>
+</segment>
+</net>
 </nets>
 </sheet>
@@
 <attribute name="TOLERANCE" x="365.76" y="180.34" size="1.778" layer="96" rot="R90" display="off"/>
 </instance>
-<instance part="GND40" gate="1" x="365.76" y="162.56" smashed="yes">
-<attribute name="VALUE" x="363.22" y="160.02" size="1.778" layer="96"/>
-</instance>
 <instance part="+3V17" gate="G$1" x="411.48" y="190.5" smashed="yes">
 <attribute name="VALUE" x="408.94" y="185.42" size="1.778" layer="96" rot="R90"/>
@@
 <attribute name="TOLERANCE" x="411.48" y="180.34" size="1.778" layer="96" rot="R90" display="off"/>
 </instance>
-<instance part="GND44" gate="1" x="411.48" y="162.56" smashed="yes">
-<attribute name="VALUE" x="408.94" y="160.02" size="1.778" layer="96"/>
-</instance>
 <instance part="U$1" gate="G$1" x="50.8" y="20.32" smashed="yes">
 <attribute name="VALUE" x="53.34" y="17.78" size="1.778" layer="96"/>
@@
 <attribute name="VALUE" x="393.7" y="55.88" size="1.778" layer="96" rot="R180"/>
 </instance>
+<instance part="U$34" gate="G$1" x="355.6" y="81.28" smashed="yes" rot="R90">
+<attribute name="VALUE" x="358.14" y="78.74" size="1.778" layer="96" rot="R180"/>
+</instance>
+<instance part="GND40" gate="1" x="355.6" y="60.96" smashed="yes" rot="R270">
+<attribute name="VALUE" x="353.06" y="63.5" size="1.778" layer="96" rot="R270"/>
+</instance>
 </instances>
 <busses>
@@
 <wire x1="187.96" y1="96.52" x2="187.96" y2="99.06" width="0.1524" layer="91"/>
 </segment>
+<segment>
+<pinref part="J8" gate="A" pin="9"/>
+<wire x1="363.22" y1="60.96" x2="360.68" y2="60.96" width="0.1524" layer="91"/>
+<wire x1="360.68" y1="60.96" x2="360.68" y2="63.5" width="0.1524" layer="91"/>
+<pinref part="J8" gate="A" pin="8"/>
+<wire x1="360.68" y1="63.5" x2="363.22" y2="63.5" width="0.1524" layer="91"/>
+<wire x1="360.68" y1="60.96" x2="358.14" y2="60.96" width="0.1524" layer="91"/>
+<junction x="360.68" y="60.96"/>
+<pinref part="GND40" gate="1" pin="GND"/>
+</segment>
 </net>
 <net name="LEAK" class="0">
@@
 </segment>
 <segment>
-<wire x1="363.22" y1="73.66" x2="360.68" y2="73.66" width="0.1524" layer="91"/>
-<label x="360.68" y="73.66" size="1.27" layer="95" rot="R180" xref="yes"/>
-<pinref part="J8" gate="A" pin="4"/>
+<wire x1="363.22" y1="71.12" x2="360.68" y2="71.12" width="0.1524" layer="91"/>
+<label x="360.68" y="71.12" size="1.27" layer="95" rot="R180" xref="yes"/>
+<pinref part="J8" gate="A" pin="5"/>
 </segment>
 <segment>
-<wire x1="363.22" y1="60.96" x2="360.68" y2="60.96" width="0.1524" layer="91"/>
-<label x="360.68" y="60.96" size="1.27" layer="95" rot="R180" xref="yes"/>
-<pinref part="J8" gate="A" pin="9"/>
+<wire x1="363.22" y1="58.42" x2="360.68" y2="58.42" width="0.1524" layer="91"/>
+<label x="360.68" y="58.42" size="1.27" layer="95" rot="R180" xref="yes"/>
+<pinref part="J8" gate="A" pin="10"/>
 </segment>
 </net>
@@
 </segment>
 </net>
-<net name="UART_RX_PH" class="0">
-<segment>
-<pinref part="J4" gate="A" pin="1"/>
-<wire x1="127" y1="38.1" x2="124.46" y2="38.1" width="0.1524" layer="91"/>
-<label x="124.46" y="38.1" size="1.27" layer="95" rot="R180" xref="yes"/>
-</segment>
-</net>
-<net name="UART_TX_PH" class="0">
-<segment>
-<pinref part="J4" gate="A" pin="2"/>
-<wire x1="127" y1="35.56" x2="124.46" y2="35.56" width="0.1524" layer="91"/>
-<label x="124.46" y="35.56" size="1.27" layer="95" rot="R180" xref="yes"/>
-</segment>
-</net>
 <net name="CS_PHT" class="0">
 <segment>
@@
 </segment>
 </net>
-<net name="RREF-" class="0">
-<segment>
-<pinref part="GND44" gate="1" pin="GND"/>
-<wire x1="411.48" y1="167.64" x2="411.48" y2="165.1" width="0.1524" layer="91"/>
-<wire x1="411.48" y1="167.64" x2="406.4" y2="167.64" width="0.1524" layer="91"/>
-<label x="406.4" y="167.64" size="1.27" layer="95" rot="R180" xref="yes"/>
-</segment>
-<segment>
-<wire x1="363.22" y1="66.04" x2="360.68" y2="66.04" width="0.1524" layer="91"/>
-<label x="360.68" y="66.04" size="1.27" layer="95" rot="R180" xref="yes"/>
-<pinref part="J8" gate="A" pin="7"/>
-</segment>
-</net>
 <net name="RSENSE+" class="0">
 <segment>
@@
 </segment>
 <segment>
-<wire x1="363.22" y1="76.2" x2="360.68" y2="76.2" width="0.1524" layer="91"/>
-<label x="360.68" y="76.2" size="1.27" layer="95" rot="R180" xref="yes"/>
-<pinref part="J8" gate="A" pin="3"/>
-</segment>
-</net>
-<net name="RSENSE-" class="0">
-<segment>
-<pinref part="GND40" gate="1" pin="GND"/>
-<wire x1="365.76" y1="167.64" x2="365.76" y2="165.1" width="0.1524" layer="91"/>
-<wire x1="365.76" y1="167.64" x2="360.68" y2="167.64" width="0.1524" layer="91"/>
-<label x="360.68" y="167.64" size="1.27" layer="95" rot="R180" xref="yes"/>
-</segment>
-<segment>
-<wire x1="363.22" y1="63.5" x2="360.68" y2="63.5" width="0.1524" layer="91"/>
-<label x="360.68" y="63.5" size="1.27" layer="95" rot="R180" xref="yes"/>
-<pinref part="J8" gate="A" pin="8"/>
+<wire x1="363.22" y1="73.66" x2="360.68" y2="73.66" width="0.1524" layer="91"/>
+<label x="360.68" y="73.66" size="1.27" layer="95" rot="R180" xref="yes"/>
+<pinref part="J8" gate="A" pin="4"/>
 </segment>
 </net>
@@
 </segment>
 <segment>
-<wire x1="363.22" y1="78.74" x2="360.68" y2="78.74" width="0.1524" layer="91"/>
-<label x="360.68" y="78.74" size="1.27" layer="95" rot="R180" xref="yes"/>
-<pinref part="J8" gate="A" pin="2"/>
+<wire x1="363.22" y1="76.2" x2="360.68" y2="76.2" width="0.1524" layer="91"/>
+<label x="360.68" y="76.2" size="1.27" layer="95" rot="R180" xref="yes"/>
+<pinref part="J8" gate="A" pin="3"/>
 </segment>
 </net>
@@
 </segment>
 </net>
+<net name="UART_RX_PH" class="0">
+<segment>
+<wire x1="127" y1="35.56" x2="124.46" y2="35.56" width="0.1524" layer="91"/>
+<label x="124.46" y="35.56" size="1.27" layer="95" rot="R180" xref="yes"/>
+<pinref part="J4" gate="A" pin="2"/>
+</segment>
+</net>
+<net name="UART_TX_PH" class="0">
+<segment>
+<wire x1="127" y1="38.1" x2="124.46" y2="38.1" width="0.1524" layer="91"/>
+<label x="124.46" y="38.1" size="1.27" layer="95" rot="R180" xref="yes"/>
+<pinref part="J4" gate="A" pin="1"/>
+</segment>
+</net>
+<net name="VIN" class="0">
+<segment>
+<pinref part="U$34" gate="G$1" pin="VIN"/>
+<wire x1="358.14" y1="81.28" x2="363.22" y2="81.28" width="0.1524" layer="91"/>
+<pinref part="J8" gate="A" pin="1"/>
+</segment>
+</net>
 </nets>
 </sheet>
@@
 <attribute name="VALUE" x="337.82" y="180.34" size="1.778" layer="96" rot="R90"/>
 </instance>
+<instance part="U$35" gate="G$1" x="383.54" y="177.8" smashed="yes"/>
 </instances>
 <busses>
@@
 <junction x="370.84" y="175.26"/>
 <pinref part="U$28" gate="G$1" pin="VIN"/>
-<wire x1="381" y1="175.26" x2="381" y2="180.34" width="0.1524" layer="91"/>
+<wire x1="381" y1="175.26" x2="381" y2="177.8" width="0.1524" layer="91"/>
+<pinref part="U$35" gate="G$1" pin="P$1"/>
+<wire x1="381" y1="177.8" x2="381" y2="180.34" width="0.1524" layer="91"/>
+<junction x="381" y="177.8"/>
 </segment>
 </net>

Commit message: Coming together
Parts:
- removed C29, C30: 1.0 uF, rcl:C-USC0603
Connections:
- net +3V3: no longer C29.1, C30.1
- net GND: no longer C29.2, C30.2
Changed lines of the file:
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@@
 <part name="U$31" library="microfloat" deviceset="TEST_POINT" device=""/>
 <part name="U$32" library="microfloat" deviceset="TEST_POINT" device=""/>
-<part name="C29" library="rcl" library_urn="urn:adsk.eagle:library:334" deviceset="C-US" device="C0603" package3d_urn="urn:adsk.eagle:package:23616/2" value="1.0 uF">
-<spice>
-<pinmapping spiceprefix="C">
-<pinmap gate="G$1" pin="1" pinorder="1"/>
-<pinmap gate="G$1" pin="2" pinorder="2"/>
-</pinmapping>
-</spice>
-<attribute name="TOLERANCE" value="5%"/>
-<attribute name="VOLTAGE" value="10V"/>
-</part>
-<part name="C30" library="rcl" library_urn="urn:adsk.eagle:library:334" deviceset="C-US" device="C0603" package3d_urn="urn:adsk.eagle:package:23616/2" value="1.0 uF">
-<spice>
-<pinmapping spiceprefix="C">
-<pinmap gate="G$1" pin="1" pinorder="1"/>
-<pinmap gate="G$1" pin="2" pinorder="2"/>
-</pinmapping>
-</spice>
-<attribute name="TOLERANCE" value="5%"/>
-<attribute name="VOLTAGE" value="10V"/>
-</part>
 <part name="C31" library="rcl" library_urn="urn:adsk.eagle:library:334" deviceset="C-US" device="C0603" package3d_urn="urn:adsk.eagle:package:23616/2" value="10uF">
 <spice>
@@
 <attribute name="VALUE" x="292.1" y="241.3" size="1.778" layer="96" rot="R270"/>
 </instance>
-<instance part="C29" gate="G$1" x="414.02" y="254" smashed="yes">
-<attribute name="NAME" x="415.036" y="254.635" size="1.778" layer="95"/>
-<attribute name="VALUE" x="415.036" y="249.809" size="1.778" layer="96"/>
-<attribute name="TOLERANCE" x="414.02" y="254" size="1.778" layer="96" display="off"/>
-<attribute name="VOLTAGE" x="414.02" y="254" size="1.778" layer="96" display="off"/>
-</instance>
-<instance part="C30" gate="G$1" x="358.14" y="254" smashed="yes">
-<attribute name="NAME" x="359.156" y="254.635" size="1.778" layer="95"/>
-<attribute name="VALUE" x="359.156" y="249.809" size="1.778" layer="96"/>
-<attribute name="TOLERANCE" x="358.14" y="254" size="1.778" layer="96" display="off"/>
-<attribute name="VOLTAGE" x="358.14" y="254" size="1.778" layer="96" display="off"/>
-</instance>
 <instance part="P+10" gate="1" x="172.72" y="27.94" smashed="yes" rot="R90">
 <attribute name="VALUE" x="177.8" y="25.4" size="1.778" layer="96" rot="R180"/>
@@
 </segment>
 <segment>
-<pinref part="C29" gate="G$1" pin="2"/>
 <wire x1="375.92" y1="246.38" x2="383.54" y2="246.38" width="0.1524" layer="91"/>
 <wire x1="383.54" y1="246.38" x2="391.16" y2="246.38" width="0.1524" layer="91"/>
 <wire x1="391.16" y1="246.38" x2="398.78" y2="246.38" width="0.1524" layer="91"/>
 <wire x1="398.78" y1="246.38" x2="406.4" y2="246.38" width="0.1524" layer="91"/>
-<wire x1="406.4" y1="246.38" x2="414.02" y2="246.38" width="0.1524" layer="91"/>
-<wire x1="414.02" y1="246.38" x2="414.02" y2="248.92" width="0.1524" layer="91"/>
 <wire x1="368.3" y1="248.92" x2="368.3" y2="246.38" width="0.1524" layer="91"/>
 <wire x1="368.3" y1="246.38" x2="375.92" y2="246.38" width="0.1524" layer="91"/>
-<wire x1="368.3" y1="246.38" x2="358.14" y2="246.38" width="0.1524" layer="91"/>
-<junction x="368.3" y="246.38"/>
-<pinref part="C30" gate="G$1" pin="2"/>
-<wire x1="358.14" y1="246.38" x2="358.14" y2="248.92" width="0.1524" layer="91"/>
 <pinref part="GND18" gate="1" pin="GND"/>
 <junction x="375.92" y="246.38"/>
@@
 <pinref part="C68" gate="G$1" pin="2"/>
 <wire x1="406.4" y1="248.92" x2="406.4" y2="246.38" width="0.1524" layer="91"/>
-<junction x="406.4" y="246.38"/>
 <pinref part="C7" gate="G$1" pin="2"/>
 <pinref part="C64" gate="G$1" pin="2"/>
@@
 <wire x1="340.36" y1="261.62" x2="368.3" y2="261.62" width="0.1524" layer="91"/>
 <pinref part="U3" gate="A" pin="VL"/>
-<wire x1="340.36" y1="256.54" x2="358.14" y2="256.54" width="0.1524" layer="91"/>
-<wire x1="358.14" y1="256.54" x2="368.3" y2="256.54" width="0.1524" layer="91"/>
+<wire x1="340.36" y1="256.54" x2="368.3" y2="256.54" width="0.1524" layer="91"/>
 <wire x1="368.3" y1="256.54" x2="368.3" y2="261.62" width="0.1524" layer="91"/>
 <junction x="368.3" y="261.62"/>
 <pinref part="+3V10" gate="G$1" pin="+3V3"/>
 <wire x1="368.3" y1="266.7" x2="368.3" y2="261.62" width="0.1524" layer="91"/>
-<pinref part="C29" gate="G$1" pin="1"/>
-<wire x1="414.02" y1="261.62" x2="414.02" y2="256.54" width="0.1524" layer="91"/>
 <wire x1="368.3" y1="261.62" x2="398.78" y2="261.62" width="0.1524" layer="91"/>
-<pinref part="C30" gate="G$1" pin="1"/>
-<junction x="358.14" y="256.54"/>
 <pinref part="C67" gate="G$1" pin="1"/>
 <wire x1="398.78" y1="261.62" x2="406.4" y2="261.62" width="0.1524" layer="91"/>
-<wire x1="406.4" y1="261.62" x2="414.02" y2="261.62" width="0.1524" layer="91"/>
 <wire x1="398.78" y1="256.54" x2="398.78" y2="261.62" width="0.1524" layer="91"/>
 <junction x="398.78" y="261.62"/>
 <pinref part="C68" gate="G$1" pin="1"/>
 <wire x1="406.4" y1="256.54" x2="406.4" y2="261.62" width="0.1524" layer="91"/>
-<junction x="406.4" y="261.62"/>
 <pinref part="C7" gate="G$1" pin="1"/>
 <junction x="368.3" y="256.54"/>

Commit message: home stretch
Parts:
- C36, C47: device rcl:C-USC0603 -> rcl:C-USC0805
Changed lines of the file:
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@@
 <attribute name="VOLTAGE" value="10V"/>
 </part>
-<part name="C36" library="rcl" library_urn="urn:adsk.eagle:library:334" deviceset="C-US" device="C0603" package3d_urn="urn:adsk.eagle:package:23616/2" value="10uF">
+<part name="C36" library="rcl" library_urn="urn:adsk.eagle:library:334" deviceset="C-US" device="C0805" package3d_urn="urn:adsk.eagle:package:23617/2" value="10uF">
 <spice>
 <pinmapping spiceprefix="C">
@@
 <attribute name="VOLTAGE" value="10V"/>
 </part>
-<part name="C47" library="rcl" library_urn="urn:adsk.eagle:library:334" deviceset="C-US" device="C0603" package3d_urn="urn:adsk.eagle:package:23616/2" value="10uF">
+<part name="C47" library="rcl" library_urn="urn:adsk.eagle:library:334" deviceset="C-US" device="C0805" package3d_urn="urn:adsk.eagle:package:23617/2" value="10uF">
 <spice>
 <pinmapping spiceprefix="C">

Commit message: DRC being weird
Connections:
- net RAD_BUSY: now also U9.PB23
Changed lines of the file:
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@@
+</segment>
+</net>
+<net name="RAD_BUSY" class="0">
+<segment>
+<wire x1="66.04" y1="99.06" x2="60.96" y2="99.06" width="0.1524" layer="91"/>
+<label x="60.96" y="99.06" size="1.27" layer="95" rot="R180" xref="yes"/>
+<pinref part="U9" gate="G$1" pin="PB23"/>
 </segment>
 </net>
@@
 </segment>
 </net>
-<net name="RAD_BUSY" class="0">
-<segment>
-<pinref part="U$3" gate="G$1" pin="BUSY"/>
-<wire x1="33.02" y1="83.82" x2="27.94" y2="83.82" width="0.1524" layer="91"/>
-<label x="27.94" y="83.82" size="1.27" layer="95" rot="R180" xref="yes"/>
-</segment>
-</net>
 <net name="!RESET_N" class="0">
 <segment>
@@
 </segment>
 </net>
+<net name="RAD_BUSY" class="0">
+<segment>
+<wire x1="33.02" y1="83.82" x2="27.94" y2="83.82" width="0.1524" layer="91"/>
+<label x="27.94" y="83.82" size="1.27" layer="95" rot="R180" xref="yes"/>
+<pinref part="U$3" gate="G$1" pin="BUSY"/>
+</segment>
+</net>

Commit message: 16 airwires and some weird ERC warnigns
Parts:
- removed C41: 10uF, rcl:CPOL-USE2.5-5
- removed C42: 100uF, rcl:CPOL-USE3.5-8
- removed C52, C55: 22uF, rcl:C-USC0805
- removed C56, C61, C67, C68: 0.1uF, rcl:C-USC0603
- removed J9: 1909763-1, microfloat:1909763-1
- removed L4: 10uH, RoboJackets-Inductors:INDUCTOR_0805
- removed R25: 649, rcl:R-US_R0603
- removed R26: 1k', rcl:R-US_R0603
- removed U$20, U$24, U$31: TEST_POINT, microfloat:TEST_POINT
- removed U9: ATSAMD51N20A-AUT, microfloat:ATSAMD51N20A-AUT
- added $$U$10, $$U$14, $$U$5: TEST_POINT, microfloat:TEST_POINT
- added C109, C112, C150, C154: 0.1 uF, rcl:C-USC0603
- added C111: 2.2 uF, rcl:C-USC0603
- added C113: 0.01 uF, rcl:C-USC0603
- added C131, C148: 0.1uF, rcl:C-USC0603
- added J5: JTAG-MINI, microfloat:JTAG-MINI
- added L101: FB-30Ohm, RoboJackets-Inductors:INDUCTOR_0805
- added R124: 100k, rcl:R-US_R0603
- added R127: 1k, rcl:R-US_R0603
- added U102: MAX13237EETE, microfloat:MAX13237EETE
- C1, C2, C3: value 0.1 uF -> 0.1uF
- C4: value 2.2 uF -> 0.1uF
- C5: value 0.01 uF -> 22uF; device rcl:C-USC0603 -> rcl:C-USC0805; VOLTAGE 10V -> 16V
- C6: value 0.1uF -> 100uF; device rcl:C-USC0603 -> rcl:CPOL-USE3.5-8; TOLERANCE 5% -> 20%; VOLTAGE 10V -> 25V
- C7: value 0.1uF -> 22uF; device rcl:C-USC0603 -> rcl:C-USC0805; VOLTAGE 10V -> 16V
- C8: value 0.1 uF -> 10uF; device rcl:C-USC0603 -> rcl:CPOL-USE2.5-5; TOLERANCE 5% -> 20%; VOLTAGE 10V -> 25V
- J2: value USB4105_REVA -> 1054291110; device microfloat:USB4105_REVA -> microfloat:1054291110
- J3: value 1054291110 -> USB4105_REVA; device microfloat:1054291110 -> microfloat:USB4105_REVA
- J6: value JTAG-MINI -> 1909763-1; device microfloat:JTAG-MINI -> microfloat:1909763-1
- L1: value FB-30Ohm -> 10uH; DKPN 490-1035-1-ND -> (none); TOLERANCE 25% -> 10%
- R1: value 100k -> 649; TOLERANCE 1% -> 0.1%
- R2: value 1k -> 1k'; TOLERANCE 1% -> 0.1%
- U$3: value LR62E -> TEST_POINT; device microfloat:LR62E -> microfloat:TEST_POINT
- U$6: value TEST_POINT -> LR62E; device microfloat:TEST_POINT -> microfloat:LR62E
- U1: value BME280 -> TXB0104PWR; device microfloat:BME280 -> microfloat:TXB0104PWR
- U3: value MAX13237EETE -> ATSAMD51N20A-AUT; device microfloat:MAX13237EETE -> microfloat:ATSAMD51N20A-AUT
- U5: value TXB0104PWR -> BME280; device microfloat:TXB0104PWR -> microfloat:BME280
- renumbered C10 to C119, C11 to C107, C13 to C103, C14 to C102, C15 to C130, C16 to C143, C17 to C139, C18 to C124, C19 to C134, C20 to C133, C21 to C100, C22 to C151, C23 to C155, C24 to C152, C25 to C153, C26 to C129, C27 to C125, C28 to C118, C31 to C110, C32 to C126, C33 to C122, C34 to C115, C35 to C127, C36 to C117, C37 to C114, C38 to C136, C39 to C141, C40 to C104, C43 to C120, C44 to C128, C45 to C121, C46 to C123, C47 to C142, C48 to C138, C49 to C145, C50 to C146, C51 to C147, C53 to C149, C54 to C156, C57 to C101, C58 to C106, C59 to C108, C60 to C105, C62 to C116, C63 to C132, C64 to C135, C65 to C144, C66 to C140, C9 to C137, CR1 to CR100, F1 to F104, F2 to F105, F3 to F100, F4 to F102, F5 to F101, F6 to F103, L2 to L102, L3 to L103, L5 to L104, L6 to L100, R10 to R116, R11 to R115, R12 to R130, R13 to R132, R14 to R106, R15 to R107, R16 to R105, R17 to R108, R18 to R109, R19 to R117, R20 to R113, R21 to R103, R22 to R104, R23 to R112, R24 to R110, R27 to R123, R28 to R100, R29 to R121, R3 to R122, R30 to R120, R31 to R129, R32 to R131, R33 to R101, R34 to R102, R35 to R125, R4 to R126, R5 to R128, R6 to R119, R7 to R118, R8 to R114, R9 to R111, T1 to T100, U$1 to U$100, U$19 to $$U$17, U$21 to $$U$2, U$27 to U$101, U$29 to $$U$4, U$32 to $$U$16, U$35 to $$U$11, U12 to U105, U13 to U100, U6 to U101, U7 to U103, U8 to U104
Connections:
- net !RESET: now also C148.1, J5.!RST, R124.1, U3.RESETN; no longer C6.1, J6.!RST, R1.1, U9.RESETN
- net !RESET_N: now also U3.PA22; no longer U9.PA22
- net !SX-NRESET: now also U$6.SX-NRESET, U3.PB20; no longer U$3.SX-NRESET, U9.PB20
- net +12V: now also U$12.P$1; no longer U$7.P$1
- net +3V3: now also $$U$14.P$1, C109.1, C111.1, C112.1, C113.1, C131.1, C150.1, C154.1, J2.9, J5.VCC, L101.1, R124.2, R2.2, U$6.VDD_RADIO, U1.VCCA, U102.!FORCEOFF, U102.VCC, U102.VL, U3.VDDIO, U3.VDDIOB, U5.VDD, U5.VDDIO; no longer C1.1, C2.1, C5.1, C67.1, C68.1, C7.1, C8.1, J4.9, J6.VCC, L1.1, R25.2, R26.2, U$3.VDD_RADIO, U$6.P$1, U1.VDD, U1.VDDIO, U3.!FORCEOFF, U3.VCC, U3.VL, U5.VCCA, U9.VDDIO, U9.VDDIOB
- net +5V: now also J4.5, U$9.P$1, U1.VCCB; no longer J3.5, U$31.P$1, U5.VCCB
- net +6V: now also J4.10; no longer J3.10
- net ANT_SW: now also U$6.ANT-SW, U3.PB21; no longer U$3.ANT-SW, U9.PB21
- net BATT_MEASURE: now also U3.PB08; no longer U9.PB08
- net CO2_IN: now also J4.1; no longer J3.1
- net CO2_OUT: now also U3.PB06; no longer U9.PB06
- net CS_GPS: now also U3.PA14; no longer U9.PA14
- net CS_IMU: now also U3.PA19; no longer U9.PA19
- net CS_PHT: now also U3.PC25, U5.CSB; no longer U1.CSB, U9.PC25
- net CS_RAD: now also U$6.NSS, U3.PA15; no longer U$3.NSS, U9.PA15
- net D_N: now also J3.DN1, J3.DN2, U3.PA24; no longer J2.DN1, J2.DN2, U9.PA24
- net D_P: now also J3.DP1, J3.DP2, U3.PA25; no longer J2.DP1, J2.DP2, U9.PA25
- net GND: now also $$U$5.P$1, C109.2, C111.2, C112.2, C113.2, C131.2, C148.2, C150.2, C154.2, C6.-, C8.-, J2.11, J2.12, J3.GND, J4.2, J4.3, J4.4, J4.6, J4.7, J4.8, J4.9, J5.GND@1, J5.GND@2, J6.GND, R127.1, U$3.P$1, U$6.GND, U102.EP, U102.FORCEON, U102.GND, U3.GNDANA; no longer C41.-, C42.-, C52.2, C55.2, C56.2, C6.2, C61.2, C67.2, C68.2, C8.2, J2.GND, J3.11, J3.12, J3.2, J3.3, J3.4, J3.6, J3.7, J3.8, J3.9, J6.GND@1, J6.GND@2, J9.GND, R2.1, U$20.P$1, U$24.P$1, U$3.GND, U3.EP, U3.FORCEON, U9.GND, U9.GNDANA
- net GPS_ANT: now also J6.SIG; no longer J9.SIG
- net IMU_INT: now also U3.PA20; no longer U9.PA20
- net LEAK: now also R127.2, U3.PB14; no longer R2.2, U9.PB14
- net LNA_EN: now also U3.PA23; no longer U9.PA23
- net MISO_1: now also U3.PC24, U5.SDO; no longer U1.SDO, U9.PC24
- net MISO_2: now also U$6.MISO, U3.PA18; no longer U$3.MISO, U9.PA18
- net MODEM_R_IN: now also U102.RIN, U3.PC16; no longer U3.RIN, U9.PC16
- net MODEM_T_IN: now also U102.TIN, U3.PC17; no longer U3.TIN, U9.PC17
- net MOSI_1: now also U3.PB24, U5.SDI; no longer U1.SDI, U9.PB24
- net MOSI_2: now also U$6.MOSI, U3.PA16; no longer U$3.MOSI, U9.PA16
- net N$1: now also U1.OE; no longer U5.OE
- net N$10: now also U102.V+; no longer U3.V+
- net N$17: now also C5.1, C7.1; no longer C52.1, C55.1
- net N$2: now also U102.C1+; no longer U3.C1+
- net N$25: now also L1.1, U3.VSW; no longer L4.1, U9.VSW
- net N$28: now also U$7.P$1; no longer U$12.P$1
- net N$4: now also U102.C1-; no longer U3.C1-
- net N$5: now also U102.C2+; no longer U3.C2+
- net N$6: now also U102.C2-; no longer U3.C2-
- net N$7: now also J3.CC2; no longer J2.CC2
- net N$8: now also C1.1, C2.1, U102.V-; no longer C56.1, C61.1, U3.V-
- net N$9: now also J3.CC1; no longer J2.CC1
- net PROBE: now also J2.10, J2.5; no longer J4.10, J4.5
- net RAD_BUSY: now also U$6.BUSY, U3.PB23; no longer U$3.BUSY, U9.PB23
- net READY: now also U102.READY, U3.PA21; no longer U3.READY, U9.PA21
- net RREF+: now also R2.1, U3.PB00; no longer R26.1, U9.PB00
- net RSENSE+: now also R1.1, U3.PB02; no longer R25.1, U9.PB02
- net R_OUT: now also J2.3, U102.ROUT; no longer J4.3, U3.ROUT
- net SCLK_1: now also U3.PB25, U5.SCK; no longer U1.SCK, U9.PB25
- net SCLK_2: now also U$6.SCK, U3.PA17; no longer U$3.SCK, U9.PA17
- net SD_CD: now also U3.PA06; no longer U9.PA06
- net SD_CK: now also U3.PB11; no longer U9.PB11
- net SD_CMD: now also U3.PA08; no longer U9.PA08
- net SD_DATA0: now also U3.PA09; no longer U9.PA09
- net SD_DATA1: now also U3.PA10; no longer U9.PA10
- net SD_DATA2: now also U3.PA11; no longer U9.PA11
- net SOLENOID: now also U3.PB15; no longer U9.PB15
- net SWCLK: now also J5.SWCLK/TCK, U3.PA30; no longer J6.SWCLK/TCK, U9.PA30
- net SWDIO: now also J5.SWIO/TMS, U3.PA31; no longer J6.SWIO/TMS, U9.PA31
- net TX_READY: now also U3.PB22; no longer U9.PB22
- net T_OUT: now also J2.4, U102.TOUT; no longer J4.4, U3.TOUT
- net UART_RX_CTD_A: now also U1.A2, U3.PB12; no longer U5.A2, U9.PB12
- net UART_RX_CTD_B: now also J2.6, U1.B2; no longer J4.6, U5.B2
- net UART_RX_M_A: now also U1.A4, U3.PB16; no longer U5.A4, U9.PB16
- net UART_RX_M_B: now also U1.B4; no longer U5.B4
- net UART_RX_PH: now also J2.2, U3.PA12; no longer J4.2, U9.PA12
- net UART_TX_CTD_A: now also U1.A1, U3.PB13; no longer U5.A1, U9.PB13
- net UART_TX_CTD_B: now also J2.7, U1.B1; no longer J4.7, U5.B1
- net UART_TX_M_A: now also U1.A3, U3.PB17; no longer U5.A3, U9.PB17
- net UART_TX_M_B: now also U1.B3; no longer U5.B3
- net UART_TX_PH: now also J2.1, U3.PA13; no longer J4.1, U9.PA13
- net VBATT: now also C6.+, C8.+; no longer C41.+, C42.+
- net VBATT_5V: now also $$U$10.P$1; no longer U$9.P$1
- net VBUS: now also J3.VBUS; no longer J2.VBUS
- net VCCA: now also L101.2, U3.VDDANA; no longer L1.2, U9.VDDANA
- net VCC_CORE: now also L1.2, U3.VDDCORE; no longer L4.2, U9.VDDCORE
- net XIN32: now also U3.PA00; no longer U9.PA00
- net XOUT32: now also U3.PA01; no longer U9.PA01
