File: pcb/microfloat.sch (EAGLE design)
At the start: 153 parts, among them J1 503182-1852, J2 1054291110, J3 USB4105_REVA, J4 1054291110, J5 JTAG-MINI, J6 1909763-1, J7 1054291110, J8 1054291110, T100 MMBT3906, U1 TXB0104PWR, U100 TPS54308DDCT, U101 LTC4419CMSEPBF, U102 MAX13237EETE, U103 TPS54308DDCT, U104 TPS54308DDCT, U105 TPS54308DDCT, U2 ICM-42688-P, U3 ATSAMD51N20A-AUT, U4 NEO-M8N-0, U5 BME280, Y1 ABS25-32.768KHZ-6-1-T

Commit message: Pain
Connections:
- net IMU_INT: now also U3.PC18; no longer U3.PA20
- net UART_RX_CTD_A: now also U1.A4; no longer U1.A2
- net UART_RX_CTD_B: now also U1.B4; no longer U1.B2
- net UART_RX_M_A: now also U1.A2; no longer U1.A4
- net UART_RX_M_B: now also U1.B2; no longer U1.B4
- net UART_TX_CTD_A: now also U1.A3; no longer U1.A1
- net UART_TX_CTD_B: now also U1.B3; no longer U1.B1
- net UART_TX_M_A: now also U1.A1; no longer U1.A3
- net UART_TX_M_B: now also U1.B1; no longer U1.B3
Changed lines of the file:
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@@
 <drawing>
 <settings>
-<setting alwaysvectorfont="yes"/>
+<setting alwaysvectorfont="no"/>
 <setting verticaltext="up"/>
 </settings>
@@
 </segment>
 </net>
-<net name="IMU_INT" class="0">
-<segment>
-<pinref part="U3" gate="G$1" pin="PA20"/>
-<wire x1="66.04" y1="182.88" x2="63.5" y2="182.88" width="0.1524" layer="91"/>
-<label x="63.5" y="182.88" size="1.27" layer="95" rot="R180" xref="yes"/>
-</segment>
-</net>
 <net name="BATT_MEASURE" class="0">
 <segment>
@@
 </segment>
 </net>
+<net name="IMU_INT" class="0">
+<segment>
+<wire x1="121.92" y1="195.58" x2="124.46" y2="195.58" width="0.1524" layer="91"/>
+<label x="124.46" y="195.58" size="1.27" layer="95" xref="yes"/>
+<pinref part="U3" gate="G$1" pin="PC18"/>
+</segment>
+</net>
 </nets>
 </sheet>
@@
 </segment>
 </net>
-<net name="UART_TX_CTD_A" class="0">
-<segment>
-<pinref part="U1" gate="A" pin="A1"/>
-<wire x1="241.3" y1="132.08" x2="238.76" y2="132.08" width="0.1524" layer="91"/>
-<label x="238.76" y="132.08" size="1.27" layer="95" rot="R180" xref="yes"/>
-</segment>
-</net>
-<net name="UART_RX_CTD_A" class="0">
-<segment>
-<pinref part="U1" gate="A" pin="A2"/>
-<wire x1="241.3" y1="129.54" x2="238.76" y2="129.54" width="0.1524" layer="91"/>
-<label x="238.76" y="129.54" size="1.27" layer="95" rot="R180" xref="yes"/>
-</segment>
-</net>
-<net name="UART_TX_M_A" class="0">
-<segment>
-<pinref part="U1" gate="A" pin="A3"/>
-<wire x1="241.3" y1="127" x2="238.76" y2="127" width="0.1524" layer="91"/>
-<label x="238.76" y="127" size="1.27" layer="95" rot="R180" xref="yes"/>
-</segment>
-</net>
-<net name="UART_RX_M_A" class="0">
-<segment>
-<pinref part="U1" gate="A" pin="A4"/>
-<wire x1="241.3" y1="124.46" x2="238.76" y2="124.46" width="0.1524" layer="91"/>
-<label x="238.76" y="124.46" size="1.27" layer="95" rot="R180" xref="yes"/>
-</segment>
-</net>
 <net name="UART_TX_M_B" class="0">
 <segment>
-<pinref part="U1" gate="A" pin="B3"/>
-<wire x1="281.94" y1="127" x2="284.48" y2="127" width="0.1524" layer="91"/>
-<label x="284.48" y="127" size="1.27" layer="95" xref="yes"/>
-</segment>
-<segment>
 <wire x1="398.78" y1="71.12" x2="396.24" y2="71.12" width="0.1524" layer="91"/>
 <label x="396.24" y="71.12" size="1.27" layer="95" rot="R180" xref="yes"/>
 <pinref part="J7" gate="A" pin="5"/>
 </segment>
-</net>
-<net name="UART_RX_M_B" class="0">
 <segment>
-<pinref part="U1" gate="A" pin="B4"/>
-<wire x1="281.94" y1="124.46" x2="284.48" y2="124.46" width="0.1524" layer="91"/>
-<label x="284.48" y="124.46" size="1.27" layer="95" xref="yes"/>
+<wire x1="281.94" y1="132.08" x2="284.48" y2="132.08" width="0.1524" layer="91"/>
+<label x="284.48" y="132.08" size="1.27" layer="95" xref="yes"/>
+<pinref part="U1" gate="A" pin="B1"/>
 </segment>
+</net>
+<net name="UART_RX_M_B" class="0">
 <segment>
 <wire x1="398.78" y1="73.66" x2="396.24" y2="73.66" width="0.1524" layer="91"/>
@@
 <pinref part="J7" gate="A" pin="4"/>
 </segment>
-</net>
-<net name="UART_TX_CTD_B" class="0">
 <segment>
-<pinref part="U1" gate="A" pin="B1"/>
-<wire x1="281.94" y1="132.08" x2="284.48" y2="132.08" width="0.1524" layer="91"/>
-<label x="284.48" y="132.08" size="1.27" layer="95" xref="yes"/>
+<wire x1="281.94" y1="129.54" x2="284.48" y2="129.54" width="0.1524" layer="91"/>
+<label x="284.48" y="129.54" size="1.27" layer="95" xref="yes"/>
+<pinref part="U1" gate="A" pin="B2"/>
 </segment>
+</net>
+<net name="UART_TX_CTD_B" class="0">
 <segment>
 <wire x1="127" y1="22.86" x2="124.46" y2="22.86" width="0.1524" layer="91"/>
@@
 <pinref part="J2" gate="A" pin="7"/>
 </segment>
-</net>
-<net name="UART_RX_CTD_B" class="0">
 <segment>
-<pinref part="U1" gate="A" pin="B2"/>
-<wire x1="281.94" y1="129.54" x2="284.48" y2="129.54" width="0.1524" layer="91"/>
-<label x="284.48" y="129.54" size="1.27" layer="95" xref="yes"/>
+<wire x1="281.94" y1="127" x2="284.48" y2="127" width="0.1524" layer="91"/>
+<label x="284.48" y="127" size="1.27" layer="95" xref="yes"/>
+<pinref part="U1" gate="A" pin="B3"/>
 </segment>
+</net>
+<net name="UART_RX_CTD_B" class="0">
 <segment>
 <pinref part="J2" gate="A" pin="6"/>
@@
 <label x="124.46" y="25.4" size="1.27" layer="95" rot="R180" xref="yes"/>
 </segment>
+<segment>
+<wire x1="281.94" y1="124.46" x2="284.48" y2="124.46" width="0.1524" layer="91"/>
+<label x="284.48" y="124.46" size="1.27" layer="95" xref="yes"/>
+<pinref part="U1" gate="A" pin="B4"/>
+</segment>
 </net>
 <net name="SOLENOID" class="0">
@@
 </segment>
 </net>
+<net name="UART_TX_M_A" class="0">
+<segment>
+<wire x1="241.3" y1="132.08" x2="238.76" y2="132.08" width="0.1524" layer="91"/>
+<label x="238.76" y="132.08" size="1.27" layer="95" rot="R180" xref="yes"/>
+<pinref part="U1" gate="A" pin="A1"/>
+</segment>
+</net>
+<net name="UART_RX_M_A" class="0">
+<segment>
+<wire x1="241.3" y1="129.54" x2="238.76" y2="129.54" width="0.1524" layer="91"/>
+<label x="238.76" y="129.54" size="1.27" layer="95" rot="R180" xref="yes"/>
+<pinref part="U1" gate="A" pin="A2"/>
+</segment>
+</net>
+<net name="UART_TX_CTD_A" class="0">
+<segment>
+<wire x1="241.3" y1="127" x2="238.76" y2="127" width="0.1524" layer="91"/>
+<label x="238.76" y="127" size="1.27" layer="95" rot="R180" xref="yes"/>
+<pinref part="U1" gate="A" pin="A3"/>
+</segment>
+</net>
+<net name="UART_RX_CTD_A" class="0">
+<segment>
+<wire x1="241.3" y1="124.46" x2="238.76" y2="124.46" width="0.1524" layer="91"/>
+<label x="238.76" y="124.46" size="1.27" layer="95" rot="R180" xref="yes"/>
+<pinref part="U1" gate="A" pin="A4"/>
+</segment>
+</net>
