File: pcb/microfloat.sch (EAGLE design)
At the start: 153 parts, among them J1 503182-1852, J2 1054291110, J3 USB4105_REVA, J4 1054291110, J5 JTAG-MINI, J6 1909763-1, J7 1054291110, J8 1054291110, T100 MMBT3906, U1 TXB0104PWR, U100 TPS54308DDCT, U101 LTC4419CMSEPBF, U102 MAX13237EETE, U103 TPS54308DDCT, U104 TPS54308DDCT, U105 TPS54308DDCT, U2 ICM-42688-P, U3 ATSAMD51N20A-AUT, U4 NEO-M8N-0, U5 BME280, Y1 ABS25-32.768KHZ-6-1-T

Commit message: More changes
Parts:
- removed R103: 68k, rcl:R-US_R0603
- removed R104: 43k, rcl:R-US_R0603
- removed U$100: SQ2348ES-T1_GE3, microfloat:SQ2348ES-T1_GE3
- removed U$101: GSOT04-E3-08, microfloat:GSOT04-E3-08
- removed U$12, U$13: TEST_POINT, microfloat:TEST_POINT
- added $$$$U$3, $$$$U$4, $$$$U$5, $$U$1: TEST_POINT, microfloat:TEST_POINT
- added R34: 1k', rcl:R-US_R0603
- added R35: 649, rcl:R-US_R0603
- $$U$10: value TEST_POINT -> SQ2348ES-T1_GE3; device microfloat:TEST_POINT -> microfloat:SQ2348ES-T1_GE3
- $$U$11: value TEST_POINT -> GSOT04-E3-08; device microfloat:TEST_POINT -> microfloat:GSOT04-E3-08
- C5: value 22uF -> 100uF; device rcl:C-USC0805 -> rcl:CPOL-USE3.5-8; TOLERANCE 5% -> 20%; VOLTAGE 16V -> 25V
- C6: value 100uF -> 22uF; device rcl:CPOL-USE3.5-8 -> rcl:C-USC0805; TOLERANCE 20% -> 5%; VOLTAGE 25V -> 16V
- J6: value 1909763-1 -> 1054291110; device microfloat:1909763-1 -> microfloat:1054291110
- J8: value 1054291110 -> 1909763-1; device microfloat:1054291110 -> microfloat:1909763-1
- R1: value 649 -> 68k
- R2: value 1k' -> 43k
- renumbered $$U$14 to $$U$7, $$U$16 to $$$$U$8, $$U$17 to $$$$U$6, C100 to C16, C101 to C17, C102 to C13, C103 to C14, C104 to C9, C105 to C18, C106 to C15, C107 to C10, C108 to C19, C109 to C11, C110 to C12, C111 to C26, C112 to C27, C113 to C28, C114 to C32, C115 to C36, C116 to C24, C117 to C33, C118 to C22, C119 to C25, C120 to C30, C121 to C34, C122 to C37, C123 to C39, C124 to C21, C125 to C20, C126 to C31, C127 to C35, C128 to C38, C129 to C40, C130 to C41, C131 to C29, C132 to C23, C133 to C47, C134 to C46, C135 to C51, C136 to C52, C137 to C48, C138 to C54, C139 to C42, C140 to C49, C141 to C53, C142 to C55, C143 to C56, C144 to C50, C145 to C43, C146 to C44, C147 to C45, C148 to C58, C149 to C64, C150 to C57, C151 to C60, C152 to C62, C153 to C63, C154 to C59, C155 to C61, C156 to C65, CR100 to CR1, F100 to F1, F101 to F2, F102 to F3, F103 to F4, F104 to F5, F105 to F6, L100 to L2, L101 to L4, L102 to L3, L103 to L5, L104 to L6, R100 to R3, R101 to R4, R102 to R5, R105 to R13, R106 to R14, R107 to R15, R108 to R16, R109 to R17, R110 to R12, R111 to R6, R112 to R11, R113 to R8, R114 to R7, R115 to R9, R116 to R10, R117 to R18, R118 to R21, R119 to R22, R120 to R23, R121 to R24, R122 to R19, R123 to R20, R124 to R25, R125 to R26, R126 to R30, R127 to R31, R128 to R29, R129 to R32, R130 to R27, R131 to R33, R132 to R28, T100 to T1, U$6 to $$U$3, U100 to U6, U101 to U8, U102 to U9, U103 to U7, U104 to U10, U105 to U11
Connections:
- net +12V: now also U$8.P$1; no longer U$12.P$1
- net +3V3: now also R34.2, R35.2; no longer R1.2, R2.2
- net +5V: now also $$U$5.P$1; no longer U$9.P$1
- net +6V: now also $$U$4.P$1; no longer U$8.P$1
- net GND: now also $$U$1.P$1, $$U$10.S, $$U$11.C, C5.-, C6.2, J6.11, J6.12, J6.8, J6.9, J8.GND, R2.1, U$9.P$1; no longer $$U$5.P$1, C5.2, C6.-, J6.GND, J8.11, J8.12, J8.8, J8.9, R104.1, U$100.S, U$101.C, U$13.P$1
- net GPS_ANT: now also J8.SIG; no longer J6.SIG
- net N$17: now also C6.1; no longer C5.1
- net N$21: now also R1.2; no longer R103.2
- net N$22: now also R1.1, R2.2; no longer R103.1, R104.2
- net N$24: now also $$U$10.G; no longer U$100.G
- net PROBE: now also J6.10, J6.5; no longer J8.10, J8.5
- net RREF+: now also J6.3, R34.1; no longer J8.3, R2.1
- net RSENSE+: now also J6.4, R35.1; no longer J8.4, R1.1
- net SOLENOID: now also $$U$11.A; no longer U$101.A
- net SOL_TRIG: now also $$U$10.D; no longer U$100.D
- net VBATT: now also $$$$U$5.P$1, C5.+; no longer $$U$11.P$1, C6.+
- net VBATT_5V: now also $$$$U$4.P$1; no longer $$U$10.P$1
- net VBUS: now also $$$$U$3.P$1; no longer $$U$4.P$1
- net VIN: now also J6.1; no longer J8.1

Commit message: BEEG Capacitor
Parts:
- removed C42, C64: 33uF, rcl:C-USC1206
- added C66, C67: KCM55TR7YA336MH01L, microfloat:KCM55TR7YA336MH01L
Connections:
- net GND: now also C66.1, C67.1; no longer C42.2, C64.2
- net VBATT: now also C66.2, C67.2; no longer C42.1, C64.1
Changed lines of the file:
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@@
 <part name="FRAME3" library="frames" library_urn="urn:adsk.eagle:library:229" deviceset="FRAME_B_L" device=""/>
 <part name="U11" library="microfloat" deviceset="TPS54308DDCT" device=""/>
-<part name="C64" library="rcl" library_urn="urn:adsk.eagle:library:334" deviceset="C-US" device="C1206" package3d_urn="urn:adsk.eagle:package:23618/2" value="33uF">
-<spice>
-<pinmapping spiceprefix="C">
-<pinmap gate="G$1" pin="1" pinorder="1"/>
-<pinmap gate="G$1" pin="2" pinorder="2"/>
-</pinmapping>
-</spice>
-<attribute name="TOLERANCE" value="5%"/>
-<attribute name="VOLTAGE" value="35V"/>
-</part>
 <part name="C65" library="rcl" library_urn="urn:adsk.eagle:library:334" deviceset="C-US" device="C0603" package3d_urn="urn:adsk.eagle:package:23616/2" value="100nF">
 <spice>
@@
 <part name="GND27" library="supply1" library_urn="urn:adsk.eagle:library:371" deviceset="GND" device=""/>
 <part name="U7" library="microfloat" deviceset="TPS54308DDCT" device=""/>
-<part name="C42" library="rcl" library_urn="urn:adsk.eagle:library:334" deviceset="C-US" device="C1206" package3d_urn="urn:adsk.eagle:package:23618/2" value="33uF">
-<spice>
-<pinmapping spiceprefix="C">
-<pinmap gate="G$1" pin="1" pinorder="1"/>
-<pinmap gate="G$1" pin="2" pinorder="2"/>
-</pinmapping>
-</spice>
-<attribute name="TOLERANCE" value="5%"/>
-<attribute name="VOLTAGE" value="35V"/>
-</part>
 <part name="C21" library="rcl" library_urn="urn:adsk.eagle:library:334" deviceset="C-US" device="C0603" package3d_urn="urn:adsk.eagle:package:23616/2" value="100nF">
 <spice>
@@
 <part name="GND40" library="supply1" library_urn="urn:adsk.eagle:library:371" deviceset="GND" device=""/>
 <part name="$$$$U$5" library="microfloat" deviceset="TEST_POINT" device=""/>
+<part name="C66" library="microfloat" deviceset="KCM55TR7YA336MH01L" device=""/>
+<part name="C67" library="microfloat" deviceset="KCM55TR7YA336MH01L" device=""/>
 </parts>
 <sheets>
@@
 <attribute name="VALUE" x="27.94" y="227.14" size="2.0828" layer="96" ratio="10" rot="SR0"/>
 </instance>
-<instance part="C64" gate="G$1" x="15.24" y="246.38" smashed="yes">
-<attribute name="NAME" x="16.256" y="247.015" size="1.778" layer="95"/>
-<attribute name="VALUE" x="16.256" y="242.189" size="1.778" layer="96"/>
-<attribute name="TOLERANCE" x="15.24" y="246.38" size="1.778" layer="96" display="off"/>
-<attribute name="VOLTAGE" x="15.24" y="246.38" size="1.778" layer="96" display="off"/>
-</instance>
 <instance part="C65" gate="G$1" x="63.5" y="248.92" smashed="yes" rot="R90">
 <attribute name="NAME" x="62.865" y="249.936" size="1.778" layer="95" rot="R90"/>
@@
 <attribute name="VALUE" x="302.26" y="222.06" size="2.0828" layer="96" ratio="10" rot="SR0"/>
 </instance>
-<instance part="C42" gate="G$1" x="289.56" y="241.3" smashed="yes">
-<attribute name="NAME" x="290.576" y="241.935" size="1.778" layer="95"/>
-<attribute name="VALUE" x="290.576" y="237.109" size="1.778" layer="96"/>
-<attribute name="TOLERANCE" x="289.56" y="241.3" size="1.778" layer="96" display="off"/>
-<attribute name="VOLTAGE" x="289.56" y="241.3" size="1.778" layer="96" display="off"/>
-</instance>
 <instance part="C21" gate="G$1" x="337.82" y="243.84" smashed="yes" rot="R90">
 <attribute name="NAME" x="337.185" y="244.856" size="1.778" layer="95" rot="R90"/>
@@
 </instance>
 <instance part="$$$$U$5" gate="G$1" x="383.54" y="177.8" smashed="yes"/>
+<instance part="C66" gate="G$1" x="15.24" y="243.84" smashed="yes" rot="R90">
+<attribute name="NAME" x="11.42906875" y="243.84" size="1.77843125" layer="95" rot="R90"/>
+<attribute name="VALUE" x="20.32848125" y="243.84" size="1.78096875" layer="96" rot="R90"/>
+</instance>
+<instance part="C67" gate="G$1" x="289.56" y="238.76" smashed="yes" rot="R90">
+<attribute name="NAME" x="285.74906875" y="238.76" size="1.77843125" layer="95" rot="R90"/>
+<attribute name="VALUE" x="294.64848125" y="238.76" size="1.78096875" layer="96" rot="R90"/>
+</instance>
 </instances>
 <busses>
@@
 </segment>
 <segment>
-<pinref part="C64" gate="G$1" pin="2"/>
 <wire x1="15.24" y1="241.3" x2="15.24" y2="238.76" width="0.1524" layer="91"/>
 <pinref part="GND52" gate="1" pin="GND"/>
+<pinref part="C66" gate="G$1" pin="1"/>
 </segment>
 <segment>
@@
 </segment>
 <segment>
-<pinref part="C42" gate="G$1" pin="2"/>
 <wire x1="289.56" y1="236.22" x2="289.56" y2="233.68" width="0.1524" layer="91"/>
 <pinref part="GND29" gate="1" pin="GND"/>
+<pinref part="C67" gate="G$1" pin="1"/>
 </segment>
 <segment>
@@
 <wire x1="22.86" y1="248.92" x2="15.24" y2="248.92" width="0.1524" layer="91"/>
 <wire x1="15.24" y1="248.92" x2="15.24" y2="254" width="0.1524" layer="91"/>
-<pinref part="C64" gate="G$1" pin="1"/>
-<junction x="15.24" y="248.92"/>
 <pinref part="U$22" gate="G$1" pin="VBATT"/>
+<pinref part="C66" gate="G$1" pin="2"/>
+<junction x="15.24" y="248.92"/>
 </segment>
 <segment>
@@
 <wire x1="297.18" y1="243.84" x2="289.56" y2="243.84" width="0.1524" layer="91"/>
 <wire x1="289.56" y1="243.84" x2="289.56" y2="248.92" width="0.1524" layer="91"/>
-<pinref part="C42" gate="G$1" pin="1"/>
-<junction x="289.56" y="243.84"/>
 <pinref part="U$5" gate="G$1" pin="VBATT"/>
+<pinref part="C67" gate="G$1" pin="2"/>
+<junction x="289.56" y="243.84"/>
 </segment>
 <segment>

Commit message: Changes I think
Parts:
- L2: value 13uH -> 10uH
- L3: value 12uH -> 10uH
- L6: value 6.471uH -> 3.9uH
Changed lines of the file:
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@@
 <attribute name="TOLERANCE" value="1%"/>
 </part>
-<part name="L6" library="RoboJackets-Inductors" deviceset="INDUCTOR_0805" device="" value="6.471uH">
+<part name="L6" library="RoboJackets-Inductors" deviceset="INDUCTOR_0805" device="" value="3.9uH">
 <attribute name="TOLERANCE" value="10%"/>
 </part>
@@
 <attribute name="TOLERANCE" value="1%"/>
 </part>
-<part name="L2" library="RoboJackets-Inductors" deviceset="INDUCTOR_0805" device="" value="13uH">
+<part name="L2" library="RoboJackets-Inductors" deviceset="INDUCTOR_0805" device="" value="10uH">
 <attribute name="TOLERANCE" value="10%"/>
 </part>
@@
 <attribute name="TOLERANCE" value="1%"/>
 </part>
-<part name="L3" library="RoboJackets-Inductors" deviceset="INDUCTOR_0805" device="" value="12uH">
+<part name="L3" library="RoboJackets-Inductors" deviceset="INDUCTOR_0805" device="" value="10uH">
 <attribute name="TOLERANCE" value="10%"/>
 </part>

Commit message: Last inductor to fix
Parts:
- removed $$U$10: SQ2348ES-T1_GE3, microfloat:SQ2348ES-T1_GE3
- removed $$U$3: LR62E, microfloat:LR62E
- removed $$U$4, $$U$7, U$7, U$8: TEST_POINT, microfloat:TEST_POINT
- removed C66, C67: KCM55TR7YA336MH01L, microfloat:KCM55TR7YA336MH01L
- added $$$$$$U$1, $$$$$$U$2, $$$$$$U$3, $$$$U$2: TEST_POINT, microfloat:TEST_POINT
- added C42: 0.1uF, rcl:C-USC0603
- added C64: 100nF, rcl:C-USC0603
- added U12, U13: TPS54308DDCT, microfloat:TPS54308DDCT
- C10: value 10 uF -> 10uF; device rcl:C-USC0603 -> rcl:CPOL-USE2.5-5; TOLERANCE 5% -> 20%; VOLTAGE 10V -> 25V
- C11: value 0.1 uF -> 10uF; device rcl:C-USC0603 -> rcl:C-USC0805; VOLTAGE 10V -> 35V
- C12: device rcl:C-USC0603 -> rcl:C-USC0805; VOLTAGE 10V -> 35V
- C15: value 100nF -> 1.0 uF; VOLTAGE 16V -> 10V
- C16: value 10uF -> 22uF; VOLTAGE 35V -> 16V
- C17: value 10uF -> 100nF; device rcl:C-USC0805 -> rcl:C-USC0603; VOLTAGE 35V -> 16V
- C18: value 22uF -> 10 uF; device rcl:C-USC0805 -> rcl:C-USC0603; VOLTAGE 16V -> 10V
- C2: value 0.1uF -> KCM55TR7YA336MH01L; device rcl:C-USC0603 -> microfloat:KCM55TR7YA336MH01L; TOLERANCE 5% -> (none); VOLTAGE 10V -> (none)
- C20: value 10uF -> 0.1 uF
- C21: value 100nF -> 10uF; VOLTAGE 16V -> 10V
- C22: value 10uF -> 2.2 uF
- C23: value 0.1uF -> 0.1 uF
- C24: value 0.1uF -> 0.01 uF
- C25: value 0.1uF -> 10uF; device rcl:C-USC0603 -> rcl:C-USC0805
- C26: value 2.2 uF -> 0.1uF
- C27: value 0.1 uF -> 0.1uF
- C28: value 0.01 uF -> 10uF; device rcl:C-USC0603 -> rcl:C-USC0805
- C29, C36: value 0.1uF -> 10uF
- C32, C33, C55: value 10uF -> 0.1uF; device rcl:C-USC0805 -> rcl:C-USC0603
- C35: value 0.1uF -> 100nF; VOLTAGE 10V -> 16V
- C44: value 10uF -> 22uF
- C45: value 1.0uF -> 22uF
- C46: value 22uF -> 0.1uF
- C47: value 22uF -> 4.7uF
- C5: value 100uF -> 0.1uF; device rcl:CPOL-USE3.5-8 -> rcl:C-USC0603; TOLERANCE 20% -> 5%; VOLTAGE 25V -> 10V
- C52: value 4.7uF -> 10uF; device rcl:C-USC0603 -> rcl:C-USC0805
- C53: value 0.1uF -> 8.2 pF; TOLERANCE 5% -> 0.5%
- C56: value 8.2 pF -> 10uF; TOLERANCE 0.5% -> 5%
- C57: value 0.1 uF -> 1.0uF
- C61: value 100nF -> 22uF
- C63: value 22uF -> 0.1 uF
- C8: value 10uF -> 100uF; device rcl:CPOL-USE2.5-5 -> rcl:CPOL-USE3.5-8
- C9: value 1.0 uF -> KCM55TR7YA336MH01L; device rcl:C-USC0603 -> microfloat:KCM55TR7YA336MH01L; TOLERANCE 5% -> (none); VOLTAGE 10V -> (none)
- J6: value 1054291110 -> 1909763-1; device microfloat:1054291110 -> microfloat:1909763-1
- J8: value 1909763-1 -> 1054291110; device microfloat:1909763-1 -> microfloat:1054291110
- L1, L2, L3: device RoboJackets-Inductors:INDUCTOR_0805 -> microfloat:78438357100
- L5, L6: device RoboJackets-Inductors:INDUCTOR_0805 -> microfloat:SRR3818A-3R9Y
- R1: value 68k -> 100k; TOLERANCE 0.1% -> 1%
- R11: value 910k -> 82k
- R12: value 82k -> 5.1k
- R13: value 100k -> 910k; TOLERANCE 1% -> 0.1%
- R14: value 10k -> 390k; TOLERANCE 1% -> 0.1%
- R15: value 10k -> 5.1k; TOLERANCE 1% -> 0.1%
- R16: value 100k -> 13.7k
- R19: value 100k -> 150k; TOLERANCE 1% -> 0.1%
- R2: value 43k -> 100k; TOLERANCE 0.1% -> 1%
- R20: value 10 -> 100k; TOLERANCE 1% -> 0.1%
- R21: value 150k -> 100k
- R22: value 100k -> 560k
- R23: TOLERANCE 0.1% -> 1%
- R24: value 560k -> 10; TOLERANCE 0.1% -> 1%
- R27: value 100k -> 1k
- R28: value 22k -> 1k
- R3: value 100k -> 11k
- R30, R31: value 1k -> 100k
- R32: value 100k -> 5.23k
- R33: value 5.23k -> 22k
- R4: value 100k -> 68k; TOLERANCE 1% -> 0.1%
- R5: value 11k -> 43k; TOLERANCE 1% -> 0.1%
- R6: value 5.1k -> 100k; TOLERANCE 0.1% -> 1%
- R7: value 5.1k -> 10k; TOLERANCE 0.1% -> 1%
- R8: value 390k -> 10k; TOLERANCE 0.1% -> 1%
- R9: value 13.7k -> 100k
- U11: value TPS54308DDCT -> SQ2348ES-T1_GE3; device microfloat:TPS54308DDCT -> microfloat:SQ2348ES-T1_GE3
- U2: value ICM-42688-P -> LR62E; device microfloat:ICM-42688-P -> microfloat:LR62E
- U3: value ATSAMD51N20A-AUT -> ICM-42688-P; device microfloat:ATSAMD51N20A-AUT -> microfloat:ICM-42688-P
- U4: value NEO-M8N-0 -> ATSAMD51N20A-AUT; device microfloat:NEO-M8N-0 -> microfloat:ATSAMD51N20A-AUT
- U5: value BME280 -> NEO-M8N-0; device microfloat:BME280 -> microfloat:NEO-M8N-0
- U6: value TPS54308DDCT -> BME280; device microfloat:TPS54308DDCT -> microfloat:BME280
- renumbered $$$$U$6 to $$$$$$U$5, $$$$U$8 to $$$$$$U$4, $$U$11 to D1, U$9 to U$6
Connections:
- net !RESET: now also U4.RESETN; no longer U3.RESETN
- net !RESET_N: now also U4.PA22, U5.RESET_N; no longer U3.PA22, U4.RESET_N
- net !SX-NRESET: now also U2.SX-NRESET, U4.PB20; no longer $$U$3.SX-NRESET, U3.PB20
- net +12V: now also $$U$5.P$1; no longer U$8.P$1
- net +3V3: now also $$$$U$5.P$1, C15.1, C18.1, C20.1, C22.1, C23.1, C24.1, C25.1, C42.1, C46.1, C5.1, C55.1, C56.1, C63.1, R1.1, R10.2, R6.2, R7.2, R8.2, R9.2, U2.VDD_RADIO, U3.VDD, U4.VDDIO, U4.VDDIOB, U5.VCC, U6.VDD, U6.VDDIO; no longer $$U$3.VDD_RADIO, $$U$7.P$1, C10.1, C11.1, C27.1, C29.1, C3.1, C30.1, C35.1, C36.1, C43.1, C44.1, C45.1, C51.1, C9.1, R13.2, R14.2, R15.2, R16.2, R17.2, R3.1, U2.VDD, U2.VDDIO, U3.VDDIOB, U4.VCC, U5.VDD, U5.VDDIO
- net +5V: now also $$$$U$4.P$1, C21.1, U12.VIN; no longer $$U$5.P$1, C12.1, U10.VIN
- net +6V: now also $$$$U$3.P$1; no longer $$U$4.P$1
- net ANT_SW: now also U2.ANT-SW, U4.PB21; no longer $$U$3.ANT-SW, U3.PB21
- net BATT_MEASURE: now also R21.2, R22.1, U4.PB08; no longer R23.2, R24.1, U3.PB08
- net CO2_IN: now also R20.2; no longer R22.2
- net CO2_OUT: now also R19.2, R20.1, U4.PB06; no longer R21.2, R22.1, U3.PB06
- net CS_GPS: now also U4.PA14, U5.SDA/SPI_CS_N; no longer U3.PA14, U4.SDA/SPI_CS_N
- net CS_IMU: now also U3.AP_CS, U4.PA19; no longer U2.AP_CS, U3.PA19
- net CS_PHT: now also U4.PC25, U6.CSB; no longer U3.PC25, U5.CSB
- net CS_RAD: now also U2.NSS, U4.PA15; no longer $$U$3.NSS, U3.PA15
- net D_N: now also U4.PA24; no longer U3.PA24
- net D_P: now also U4.PA25; no longer U3.PA25
- net GND: now also $$$$U$2.P$1, C10.-, C15.2, C2.1, C21.2, C23.2, C24.2, C25.2, C42.2, C5.2, C61.2, C9.1, J6.GND, J8.11, J8.12, J8.8, J8.9, R11.1, R12.2, R15.1, R16.1, R3.1, R32.1, U11.S, U12.GND, U13.GND, U3.RESV_10, U3.RESV_11, U3.RESV_2, U3.RESV_3, U3.RESV_7, U4.GNDANA, U5.D_SEL, U5.VDD_USB; no longer $$U$10.S, $$U$3.GND, C10.2, C17.2, C2.2, C27.2, C30.2, C35.2, C43.2, C5.-, C66.1, C67.1, C9.2, J6.11, J6.12, J6.8, J6.9, J8.GND, R12.1, R2.1, R31.1, R6.2, R7.1, R9.1, U$3.P$1, U11.GND, U2.RESV_10, U2.RESV_11, U2.RESV_2, U2.RESV_3, U2.RESV_7, U3.GNDANA, U4.D_SEL, U4.VDD_USB
- net GPS_ANT: now also J6.SIG, U5.RF_IN; no longer J8.SIG, U4.RF_IN
- net IMU_INT: now also U3.INT1/INT, U4.PC18; no longer U2.INT1/INT, U3.PC18
- net LEAK: now also R28.2, U4.PB14; no longer R31.2, U3.PB14
- net LNA_EN: now also U4.PA23, U5.LNA_EN; no longer U3.PA23, U4.LNA_EN
- net MISO_1: now also U4.PC24, U5.TXD/SPI_MISO, U6.SDO; no longer U3.PC24, U4.TXD/SPI_MISO, U5.SDO
- net MISO_2: now also U2.MISO, U3.AP_SDO/AP_AD0, U4.PA18; no longer $$U$3.MISO, U2.AP_SDO/AP_AD0, U3.PA18
- net MODEM_R_IN: now also U4.PC16; no longer U3.PC16
- net MODEM_T_IN: now also U4.PC17; no longer U3.PC17
- net MOSI_1: now also U4.PB24, U5.RXD/SPI_MOSI, U6.SDI; no longer U3.PB24, U4.RXD/SPI_MOSI, U5.SDI
- net MOSI_2: now also U2.MOSI, U3.AP_SDA/AP_SDIO/AP_SDI, U4.PA16; no longer $$U$3.MOSI, U2.AP_SDA/AP_SDIO/AP_SDI, U3.PA16
- net N$1: now also R1.2; no longer R3.2
- net N$10: now also C54.1; no longer C49.1
- net N$11: now also C35.1, U10.BOOT; no longer C21.1, U7.BOOT
- net N$12: now also C35.2, L1.P$2, U10.SW; no longer C21.2, L3.1, U7.SW
- net N$13: now also R16.2, R17.1, U10.FB; no longer R10.1, R9.2, U7.FB
- net N$14: now also C64.1, U12.BOOT; no longer C61.1, U10.BOOT
- net N$15: now also C64.2, L5.P$2, U12.SW; no longer C61.2, L5.1, U10.SW
- net N$16: now also R31.1, R33.2, U12.FB; no longer R27.1, R28.2, U10.FB
- net N$17: now also L6.P$1, R30.2; no longer L6.2, R32.2
- net N$18: now also C16.1, L3.P$1, R2.2; no longer C18.1, L2.2, R4.2
- net N$19: now also C44.1, C45.1, L1.P$1, R17.2; no longer C46.1, C47.1, L3.2, R10.2
- net N$2: now also C43.1; no longer C23.1
- net N$20: now also C61.1, L5.P$1, R31.2; no longer C63.1, L5.2, R27.2
- net N$21: now also R14.1, R4.2; no longer R1.2, R8.1
- net N$22: now also R4.1, R5.2; no longer R1.1, R2.2
- net N$23: now also R11.2, R13.1; no longer R11.1, R12.2
- net N$24: now also R24.1, U11.G; no longer $$U$10.G, R20.1
- net N$25: now also L2.P$2, U4.VSW; no longer L1.1, U3.VSW
- net N$26: now also C36.1, R14.2; no longer C20.1, R8.2
- net N$28: now also U$3.P$1; no longer U$7.P$1
- net N$3: now also R27.1; no longer R30.1
- net N$32: now also U5.V_BCKP; no longer U4.V_BCKP
- net N$35: now also U13.BOOT; no longer U11.BOOT
- net N$36: now also L6.P$2, U13.SW; no longer L6.1, U11.SW
- net N$37: now also R30.1, R32.2, U13.FB; no longer R32.1, R33.2, U11.FB
- net N$38: now also C17.1, U7.BOOT; no longer C15.1, U6.BOOT
- net N$39: now also C17.2, L3.P$2, U7.SW; no longer C15.2, L2.1, U6.SW
- net N$4: now also C43.2; no longer C23.2
- net N$40: now also R2.1, R3.2, U7.FB; no longer R4.1, R5.2, U6.FB
- net N$5: now also C27.1, C30.1; no longer C24.1, C25.1
- net N$6: now also C27.2, C30.2; no longer C24.2, C25.2
- net N$7: now also R15.2; no longer R7.2
- net N$8: now also C3.1; no longer C2.1
- net N$9: now also R12.1; no longer R6.1
- net PROBE: now also J8.10, J8.5, R27.2; no longer J6.10, J6.5, R30.2
- net RAD_BUSY: now also U2.BUSY, U4.PB23; no longer $$U$3.BUSY, U3.PB23
- net READY: now also U4.PA21; no longer U3.PA21
- net RREF+: now also J8.3, U4.PB00; no longer J6.3, U3.PB00
- net RSENSE+: now also J8.4, U4.PB02; no longer J6.4, U3.PB02
- net SCLK_1: now also U4.PB25, U5.SCL/SPI_CLK, U6.SCK; no longer U3.PB25, U4.SCL/SPI_CLK, U5.SCK
- net SCLK_2: now also U2.SCK, U3.AP_SCL/AP_SCLK, U4.PA17; no longer $$U$3.SCK, U2.AP_SCL/AP_SCLK, U3.PA17
- net SD_CD: now also R7.1, U4.PA06; no longer R14.1, U3.PA06
- net SD_CK: now also U4.PB11; no longer U3.PB11
- net SD_CMD: now also R8.1, U4.PA08; no longer R15.1, U3.PA08
- net SD_DATA0: now also R9.1, U4.PA09; no longer R16.1, U3.PA09
- net SD_DATA1: now also R10.1, U4.PA10; no longer R17.1, U3.PA10
- net SD_DATA2: now also R6.1, U4.PA11; no longer R13.1, U3.PA11
- net SOLENOID: now also R23.2, R24.2, U4.PB15; no longer R19.2, R20.2, U3.PB15
- net SOL_TRIG: now also U11.D; no longer $$U$10.D
- net SWCLK: now also U4.PA30; no longer U3.PA30
- net SWDIO: now also U4.PA31; no longer U3.PA31
- net TX_READY: now also U4.PB22, U5.EXTINT; no longer U3.PB22, U4.EXTINT
- net UART_RX_CTD_A: now also U4.PB12; no longer U3.PB12
- net UART_RX_M_A: now also U4.PB16; no longer U3.PB16
- net UART_RX_PH: now also U4.PA12; no longer U3.PA12
- net UART_TX_CTD_A: now also U4.PB13; no longer U3.PB13
- net UART_TX_M_A: now also U4.PB17; no longer U3.PB17
- net UART_TX_PH: now also U4.PA13; no longer U3.PA13
- net VBATT: now also $$$$$$U$3.P$1, C10.+, C11.1, C12.1, C2.2, C9.2, R22.2, U10.VIN, U13.VIN; no longer $$$$U$5.P$1, C16.1, C17.1, C5.+, C66.2, C67.2, R24.2, U11.VIN, U6.VIN
- net VBATT_5V: now also $$$$$$U$2.P$1, C29.1, R13.2; no longer $$$$U$4.P$1, C22.1, R11.2
- net VBUS: now also $$$$$$U$1.P$1; no longer $$$$U$3.P$1
- net VCCA: now also C49.1, C52.1, U4.VDDANA; no longer C54.1, C55.1, U3.VDDANA
- net VCC_CORE: now also C47.1, C51.1, L2.P$1, U4.VDDCORE; no longer C52.1, C53.1, L1.2, U3.VDDCORE
- net VIN: now also J8.1; no longer J6.1
- net XIN32: now also C53.1, U4.PA00; no longer C56.1, U3.PA00
- net XOUT32: now also U4.PA01; no longer U3.PA01
Other:
- moved on the sheet: C12, C16, C17, C21, C23, C24, C27, C3, C31, C32, C33, C34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

Commit message: WEEEEEEEEEEEEEEEE
Parts:
- C47: value 4.7uF -> 0.1uF
- C51: value 0.1uF -> 10uF; device rcl:C-USC0603 -> rcl:C-USC0805
- C52: value 10uF -> 8.2 pF; device rcl:C-USC0805 -> rcl:C-USC0603; TOLERANCE 5% -> 0.5%
- C53: value 8.2 pF -> 0.1uF; TOLERANCE 0.5% -> 5%
- C54: value 0.1uF -> 4.7uF
- L3: value 10uH -> FB-30Ohm; device microfloat:78438357100 -> RoboJackets-Inductors:INDUCTOR_0805; DKPN (none) -> 490-1035-1-ND; TOLERANCE 10% -> 25%
- L4: value FB-30Ohm -> 10uH; device RoboJackets-Inductors:INDUCTOR_0805 -> microfloat:78438357100; DKPN 490-1035-1-ND -> (none); TOLERANCE 25% -> 10%
- renumbered U$6 to $$U$3
Connections:
- net +3V3: now also L3.1; no longer L4.1
- net GND: now also C48.2; no longer C47.2
- net N$10: now also C49.1, C53.1; no longer C50.1, C54.1
- net N$18: now also L2.P$1; no longer L3.P$1
- net N$2: now also C47.1; no longer C48.1
- net N$25: now also L4.P$2; no longer L2.P$2
- net N$39: now also L2.P$2; no longer L3.P$2
- net N$4: now also C47.2; no longer C48.2
- net VCCA: now also C48.1, C51.1, L3.2; no longer C49.1, C52.1, L4.2
- net VCC_CORE: now also C50.1, C54.1, L4.P$1; no longer C47.1, C51.1, L2.P$1
- net XIN32: now also C52.1; no longer C53.1
Other:
- moved on the sheet: C51, C52

Commit message: Test poitns are cool
Parts:
- added $$$$$$U$6: TEST_POINT, microfloat:TEST_POINT
Connections:
- net VIN: now also $$$$$$U$6.P$1
Changed lines of the file:
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@@
 <part name="C9" library="microfloat" deviceset="KCM55TR7YA336MH01L" device=""/>
 <part name="C2" library="microfloat" deviceset="KCM55TR7YA336MH01L" device=""/>
+<part name="$$$$$$U$6" library="microfloat" deviceset="TEST_POINT" device=""/>
 </parts>
 <sheets>
@@
 <attribute name="VALUE" x="294.64848125" y="238.76" size="1.78096875" layer="96" rot="R90"/>
 </instance>
+<instance part="$$$$$$U$6" gate="G$1" x="342.9" y="177.8" smashed="yes"/>
 </instances>
 <busses>
@@
 <segment>
 <pinref part="U$18" gate="G$1" pin="VIN"/>
-<wire x1="340.36" y1="180.34" x2="340.36" y2="175.26" width="0.1524" layer="91"/>
+<wire x1="340.36" y1="180.34" x2="340.36" y2="177.8" width="0.1524" layer="91"/>
 <pinref part="F4" gate="G$1" pin="2"/>
+<wire x1="340.36" y1="177.8" x2="340.36" y2="175.26" width="0.1524" layer="91"/>
 <wire x1="340.36" y1="175.26" x2="342.9" y2="175.26" width="0.1524" layer="91"/>
+<pinref part="$$$$$$U$6" gate="G$1" pin="P$1"/>
+<junction x="340.36" y="177.8"/>
 </segment>
 </net>

Commit message: And another one bites the dust
Parts:
- removed U$3: TEST_POINT, microfloat:TEST_POINT
Connections:
- removed net N$28: U$3.P$1, U8.V2ON
Changed lines of the file:
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@@
 <part name="$$$$U$3" library="microfloat" deviceset="TEST_POINT" device=""/>
 <part name="$$$$$$U$2" library="microfloat" deviceset="TEST_POINT" device=""/>
-<part name="U$3" library="microfloat" deviceset="TEST_POINT" device=""/>
 <part name="$$$$U$2" library="microfloat" deviceset="TEST_POINT" device=""/>
 <part name="$$$$$$U$5" library="microfloat" deviceset="TEST_POINT" device=""/>
@@
 <instance part="$$$$U$3" gate="G$1" x="251.46" y="264.16" smashed="yes"/>
 <instance part="$$$$$$U$2" gate="G$1" x="383.54" y="259.08" smashed="yes"/>
-<instance part="U$3" gate="G$1" x="241.3" y="132.08" smashed="yes"/>
 <instance part="$$$$U$2" gate="G$1" x="284.48" y="177.8" smashed="yes"/>
 <instance part="$$$$$$U$5" gate="G$1" x="284.48" y="172.72" smashed="yes"/>
@@
 </segment>
 </net>
-<net name="N$28" class="0">
-<segment>
-<pinref part="U$3" gate="G$1" pin="P$1"/>
-<pinref part="U8" gate="A" pin="V2ON"/>
-<wire x1="238.76" y1="132.08" x2="233.68" y2="132.08" width="0.1524" layer="91"/>
-</segment>
-</net>
